File: PCB/Controller/_autosave-Controller.kicad_pcb (KiCad board)
At the start: 4 copper layers, 150 x 110 mm, 284 parts, among them CN1 XT60PW_M, CN2 XT60PW_F, CN4 XT60PW_F, CN5 XT60PW_F, CN6 XT60PW_F, J1 Conn_02x07_Odd_Even, J10 Conn_01x03_Pin, J12 Conn_02x02_Top_Bottom, J13 Conn_01x14_Pin, J14 Conn_01x06_Pin, J15 Conn_01x14_Socket, J16 Conn_01x06_Socket, J17 Conn_01x06_Socket, J18 Conn_01x14_Pin, J19 Conn_01x06_Pin, J2 Conn_01x02_Pin, J20 Conn_01x14_Socket, J21 Conn_02x04_Odd_Even, J5 Conn_01x03_Pin, J6 Conn_01x03_Pin, J7 Conn_01x03_Pin, J8 Conn_01x03_Pin, J9 Conn_01x02_Pin, Q1 CSD16340Q3, Q10 LBSS138LT1G, Q2 CSD16340Q3, Q3 CSD16340Q3, Q5 CSD16340Q3, Q7 LBSS138LT1G, Q8 LBSS138LT1G, Q9 LBSS138LT1G, SW1 TS-1088-AR02016, SW10 DSIC03LSGET, SW11 TS-1088-AR02016, SW12 TS-1088-AR02016, SW13 MK-11C04-G013, SW14 DSIC03LSGET, SW2 TS-1088-AR02016, SW3 TS-1088-AR02016, SW4 TS-1088-AR02016, SW5 TS-1088-AR02016, SW6 TS-1088-AR02016, SW7 TS-1088-AR02016, SW8 TS-1088-AR02016, SW9 TS-1088-AR02016, U1 STM32F765VGTx, U11 INA226AQDGSRQ1, U12 LMR51430, U13 100uF, U14 BME280, U15 S322527M20PF10PPM, U16 TXB0108RGYR, U17 TX5813, U18 100uF, U19 TPS259850RQPR, U2 BNO080, U20 LD1117D33TR, U3 BMP580, U4 XAL5050-562MEC, U5 MAX7456EUI, U6 SMA_Conn, U7 TPS55289RYQR, U8 XAL7070-472MEC, U9 TPS630701RNMT, X1 X322525MOB4SI, X2 Q13FC1350000400

Commit message: Update
Parts:
- moved U10 14.8 mm to (204.5, 95.1)
- moved C13 10.5 mm to (165.2, 133.8)
- moved BUZ1 6.96 mm to (187.2, 73.2), turned to 135 degrees
- moved C12 4.49 mm to (170.8, 128.2)
- moved C11 0.95 mm to (175.0, 133.0)
- moved C10 0.89 mm to (169.2, 136.8)
- moved C78 0.89 mm to (170.0, 136.0)
- moved R73 0.50 mm to (196.2, 149.5)
- moved R74 0.50 mm to (183.8, 149.5)
- moved R75 0.25 mm to (182.0, 149.5)
Connections:
- J1 pad 1: VBAT -> VSYS
- J1 pad 3: VBUS -> VSYS
- J1 pad 5: VMOTORS -> VSYS
- LED3 pad 2: INA_ALERT -> INA_ALERT_T
- R6 pad 1: INA_ALERT -> INA_ALERT_T
Routing:
- net +3.3V: track 84.4 -> 371.2 mm, vias 2 -> 26
- net +5V: track 0.00 -> 189.2 mm, vias 0 -> 8
- net VSYS: track 0.00 -> 176.2 mm, vias 0 -> 1
- net +12V: track 0.00 -> 156.1 mm, vias 0 -> 2
- net INA_ALERT_T: track 0.00 -> 98.4 mm, vias 0 -> 2
- net MAIN_SCK_T: track 15.2 -> 110.2 mm, vias 2 -> 4
- net MAIN_SDA_T: track 18.1 -> 112.5 mm, vias 2 -> 4
- net VOLTAGE_ADC_T: track 0.00 -> 86.9 mm, vias 0 -> 2
- net VBAT: track 0.00 -> 82.7 mm, vias 0 -> 2
- net VMOTORS: track 0.00 -> 79.9 mm, vias 0 -> 2
- net BUTTON_LEFT: track 0.00 -> 63.9 mm, vias 0 -> 2
- net DISP_E: track 0.00 -> 61.6 mm, vias 0 -> 2
- net BUTTON_DECREASE: track 0.00 -> 60.4 mm, vias 0 -> 2
- net DISP_DP: track 0.00 -> 59.8 mm, vias 0 -> 2
- net BUTTON_INCREASE: track 0.00 -> 56.4 mm, vias 0 -> 2
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- added copper zone on F.Cu, net +3.3V
- added copper zone on B.Cu, net GND
- added copper zone on F.Cu, net GND
- added copper zone on In1.Cu, net GND
- added copper zone on In2.Cu, net GND
- added copper zone on F.Cu, net Net-(U12-SW)
Other:
- board size 150 x 110 mm -> 150 x 110.5 mm
