File: PCB/Controller/Controller.kicad_sch (KiCad schematic)
At the start: 22 parts, among them CN1 XT60PW_M, CN2 XT60PW_F, CN3 Camera Conn, J1 Screw_Terminal_01x02, SW1 TS-1088-AR02016, U1 STM32F765VGTx, U10 BQ40Z50RSMR-R2, U11 INA226AQDGSRQ1, U12 LMR51430, U2 BNO080, U3 BMP580, U4 BQ25703ARSNR, U5 MAX7456EUI, U6 SMA_Conn, U7 AL8871QT16E-13, U8 STUSB4500QTR, U9 TPS630701RNMT

Commit message: Update
Parts:
- removed J1: Screw_Terminal_01x02, symbol Connector:Screw_Terminal_01x02
- removed U10: BQ40Z50RSMR-R2, LCSC:VQFN-32_L4.0-W4.0-P0.40-TL-EP1.4_2, symbol LCSC:BQ40Z50RSMR-R2
- removed U4: BQ25703ARSNR, LCSC:VQFN-32_L4.0-W4.0-P0.40-TL-EP, symbol LCSC:BQ25703ARSNR
- removed U7: AL8871QT16E-13, LCSC:TSSOP-16_L5.0-W4.4-P0.65-LS6.4-BL-EP-2, symbol LCSC:AL8871QT16E-13
- removed U8: STUSB4500QTR, Package_DFN_QFN:QFN-24-1EP_4x4mm_P0.5mm_EP2.7x2.7mm, symbol Interface_USB:STUSB4500QTR
- added C1: 0.1uF, Capacitor_SMD:C_0603_1608Metric, symbol Device:C
- added C10: 2.2uF, symbol Device:C
- added C11, C14, C15: 0.1uF, symbol Device:C
- added C12, C13, C16, C19, C20, C21, C22: 22uF, symbol Device:C
- added C17: 4.7uF, symbol Device:C
- added C18: 22nF, symbol Device:C
- added C2: 100nF, Capacitor_SMD:C_0402_1005Metric, symbol Device:C
- added C23: 3300pF, symbol Device:C
- added C24: 330pF, symbol Device:C
- added C25: 47uF, lcsc:CAP-SMD_BD6.3-L6.6-W6.6-LS7.2-FD, symbol LCSC:RVT1E470M060547UF25V
- added C26, C27: 100nF, symbol Device:C
- added C3, C6: 10uF, Capacitor_SMD:C_0603_1608Metric, symbol Device:C
- added C4, C5: 10uF, Capacitor_SMD:C_0805_2012Metric, symbol Device:C
- added C7, C8, C9: 22uF, Capacitor_SMD:C_0805_2012Metric, symbol Device:C
- added CN4, CN5, CN6: XT60PW_F, Connector_AMASS:AMASS_XT60PW-F_1x02_P7.20mm_Horizontal, symbol LCSC:XT60PW-F_C428722
- added D1, D2: SS34, Diode_SMD:D_SMA, symbol Diode:SS34
- added J3, J4: Conn_01x06_Pin, symbol Connector:Conn_01x06_Pin
- added L1: XFL4020-152MEC, LCSC:IND-SMD_L4.0-W4.0-A, symbol LCSC:XFL4020-152MEC
- added P1: WJ127-5.0-2P, LCSC:CONN-TH_2P-P5.00_CPC3703CTR, symbol LCSC:WJ127-5.0-2P
- added Q1, Q2, Q3, Q4, Q5, Q6: CSD16340Q3, LCSC:VSON-CLIP-8_L3.3-W3.3-P0.65-BL, symbol LCSC:CSD16340Q3
- added R10: 22.1K, symbol Device:R
- added R11: 68K, symbol Device:R
- added R12, R7: 10K, symbol Device:R
- added R13, R14: 56K, symbol Device:R
- added R15: MS122WF100MT4E, lcsc:R2512, symbol LCSC:MS122WF100MT4E
- added R16: 4.7K, symbol Device:R
- added R17, R18, R19, R20, R21, R22: 33, symbol Device:R
- added R3: HOLR2725D-4W-2MR-1%, LCSC:R2725, symbol LCSC:HOLR2725D-4W-2MR-1%
- added R4, R5, R6: 1K, symbol Device:R
- added R8, R9: 100K, symbol Device:R
- added U10: RVT1E101M0607 100UF 25V, lcsc:CAP-SMD_BD6.3-L6.6-W6.6-LS7.2-FD-1, symbol LCSC:RVT1E101M0607100UF25V
- added U13: 100UF, lcsc:CAP-SMD_BD6.3-L6.6-W6.6-LS7.2-FD-1, symbol LCSC:RVT1E101M0607100UF25V
- added U4: XAL5050-562MEC, lcsc:IND-SMD_L5.5-W5.3, symbol LCSC:XAL5050-562MEC
- added U7: TPS55289RYQR, lcsc:VQFN-21_L5.0-W3.0-P0.50-TL, symbol LCSC:TPS55289RYQR
- added U8: XAL7070-472MEC, lcsc:IND-SMD_L7.5-W7.2-1, symbol LCSC:XAL7070-472MEC
- CN1: footprint lcsc:CONN-TH_XT60PW-M -> Connector_AMASS:AMASS_XT60PW-M_1x02_P7.20mm_Horizontal
- CN2: footprint lcsc:TH_2P-XT60PW-F -> Connector_AMASS:AMASS_XT60PW-F_1x02_P7.20mm_Horizontal
Connections:
- net GND: now also U11.1 (A1), U11.2 (A0), U11.7 (GND), U12.1 (GND), U9.10 (PGND), U9.15 (VSEL), U9.4 (GND), U9.6 (FB2), C1.1, C10.2, C17.1, C18.1, C2.2, C23.1, C24.1, C3.1, C4.1, C5.1, C6.1, C7.1, C8.1, C9.1, R10.2, R13.1, R14.2, R16.1, R4.1, R5.1, R6.1, U7.17 (AGND)
- net VBUS: now also D1.2 (A)
- net PGND: now reaches CN2.1
- net PGND: now also CN1.2 (+), CN1.3, CN1.4, CN2.2, CN2.4 (-), C16.1, C19.1, C20.1, C21.1, C22.1, C25.1, C27.1, CN4.1, CN4.2, CN4.4 (-), CN5.1, CN5.2, CN5.4 (-), CN6.1, CN6.2, CN6.4 (-), P1.2, Q1.1 (S), Q1.2 (S), Q1.3 (S), Q2.1 (S), Q2.2 (S), Q2.3 (S), Q3.1 (S), Q3.2 (S), Q3.3 (S), Q4.1 (S), Q4.2 (S), Q4.3 (S), Q5.1 (S), Q5.2 (S), Q5.3 (S), Q6.1 (S), Q6.2 (S), Q6.3 (S), U13.1, U7.9 (PGND)
- net VMOTORS: now reaches CN2.3 (+)
- net VMOTORS: now also U11.9 (VIN-), CN4.3 (+), CN5.3 (+), CN6.3 (+), D2.2 (A), R3.1
- net VBAT: now reaches CN1.1 (-)
- net VBAT: now also U11.10 (VIN+), U11.8 (VBUS), P1.1, R3.2
- net at U12.2 (SW): now also C11.2, U4.1
- net VSYS: now reaches U12.3 (VIN)
- net VSYS: now also U12.5 (EN), U9.12 (VIN), C10.1, C16.2, C27.2, C3.2, C4.2, C5.2, D1.1 (K), D2.1 (K), R7.1, U13.2, U7.7 (VIN)
- net at U12.4 (FB): now also C12.1, C13.1, R10.1, R9.2
- net at U12.6 (CB): now also C11.1
- net INA_ALERT: now reaches U11.3 (Alert)
- net INA_ALERT: now also R6.2
- net INA_SDA: now reaches U11.4 (SDA)
- net INA_SDA: now also R4.2
- net INA_SCL: now reaches U11.5 (SCL)
- net INA_SCL: now also R5.2
- net +3.3V: now reaches U11.6 (VS+)
- net +3.3V: now also C1.2, C12.2, C13.2, R9.1, U4.2
- net at U9.1 (PS/S): now also U9.14 (EN), R7.2
- net at U9.11 (L1): now also L1.1
- net at U9.2 (PG): now also R8.1
- net at U9.3 (VAUX): now also C2.1
- net +5V: now reaches U9.5 (FB)
- net +5V: now also U9.7 (VOUT), C6.2, C7.2, C8.2, C9.2, R8.2
- net at U9.9 (L2): now also L1.2
- new net: C23.2, R12.2, U7.15 (COMP)
- new net: R11.1, R16.2, U7.14 (FB/~{INT})
- new net: C19.2, C20.2, C21.2, C22.2, C25.2, C26.2, R15.1, U7.11 (VOUT), U7.12 (ISP)
- new net: Q6.4 (G), R22.1
- new net: C14.1, U7.20 (BOOT1)
- new net: C17.2, U7.18 (VCC)
- new net: Q5.4 (G), R21.1
- new net: R13.2, U7.16 (CDC)
- new net: C24.2, R12.1
- new net: Q3.4 (G), R19.1
- new net: Q4.4 (G), R20.1
- new net: Q1.4 (G), R17.1
- new net: C15.1, U7.19 (BOOT2)
- new net: Q2.4 (G), R18.1
- new net: C18.2, U7.5 (DITH/SYNC)
- new net: R14.1, U7.6 (FSW)
- new net +12V: C26.1, J4.1 (Pin_1), J4.2 (Pin_2), J4.3 (Pin_3), J4.4 (Pin_4), J4.5 (Pin_5), J4.6 (Pin_6), R11.2, R15.2, U7.13 (ISN)
- new net BOOT1: C14.2, U7.8 (SW1), U8.2
- new net BOOT2: C15.2, U7.10 (SW2), U8.1
- new net LED1_POWER: J3.1 (Pin_1), Q1.5 (D), Q1.6 (D), Q1.7 (D), Q1.8 (D)
- new net LED1_PWM: R17.2
- new net LED2_POWER: J3.2 (Pin_2), Q2.5 (D), Q2.6 (D), Q2.7 (D), Q2.8 (D)
- new net LED2_PWM: R18.2
- new net LED3_POWER: J3.3 (Pin_3), Q5.5 (D), Q5.6 (D), Q5.7 (D), Q5.8 (D)
- new net LED3_PWM: R21.2
- new net LED4_POWER: J3.4 (Pin_4), Q3.5 (D), Q3.6 (D), Q3.7 (D), Q3.8 (D)
- new net LED4_PWM: R19.2
- new net LED5_POWER: J3.5 (Pin_5), Q4.5 (D), Q4.6 (D), Q4.7 (D), Q4.8 (D)
- new net LED5_PWM: R20.2
- new net LED6_POWER: J3.6 (Pin_6), Q6.5 (D), Q6.6 (D), Q6.7 (D), Q6.8 (D)
- new net LED6_PWM: R22.2
Other:
- moved on the sheet: CN1, CN2, CN3, Card1, LED1, SW1, U1, U11, U12, U2, U3, U5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

Commit message: Update
Parts:
- removed U10: RVT1E101M0607 100UF 25V, lcsc:CAP-SMD_BD6.3-L6.6-W6.6-LS7.2-FD-1, symbol LCSC:RVT1E101M0607100UF25V
- added C28: 22nF, Capacitor_SMD:C_0603_1608Metric, symbol Device:C
- added C29, C30, C31, C32, C33, C34, C36, C37, C38, C41: 100nF, symbol Device:C
- added C35: 10uF, symbol Device:C
- added C39, C40: 20pF, symbol Device:C
- added C42, C43: C_Polarized, symbol Device:C_Polarized
- added D3, D4, D5, D6: SS34, Diode_SMD:D_SMA, symbol Diode:SS34
- added J1, J2: Conn_01x06_Pin, symbol Connector:Conn_01x06_Pin
- added J10, J5, J6, J7, J8: Conn_01x03_Pin, symbol Connector:Conn_01x03_Pin
- added J9: Conn_01x02_Pin, symbol Connector:Conn_01x02_Pin
- added LED10, LED17, LED18, LED19: KT-0603B, lcsc:LED0603-RD, symbol LCSC:Bluelight0603
- added LED11, LED12, LED13, LED14, LED15, LED16, LED2: KT-0603YG, lcsc:LED0603-RD, symbol LCSC:XL-0603QYGC
- added LED3: KT-0603R, lcsc:LED0603-RD, symbol LCSC:KT-0603R
- added LED4, LED5, LED6, LED7, LED8, LED9: KT-0603W, lcsc:LED0603-R-RD_WHITE, symbol LCSC:0603Whitelight_C2290
- added NT1: NetTie_4, symbol Device:NetTie_4
- added NT2: NetTie_2, symbol Device:NetTie_2
- added Q10, Q7, Q8, Q9: LBSS138LT1G, lcsc:SOT-23_L2.9-W1.3-P1.90-LS2.4-BR, symbol LCSC:LBSS138LT1G
- added R23: 150K, Resistor_SMD:R_0603_1608Metric, symbol Device:R
- added R24: 47K, Resistor_SMD:R_0603_1608Metric, symbol Device:R
- added R25, R26: 2.2K, symbol Device:R
- added R27, R28, R29, R30, R31, R32, R33, R34, R35, R49, R50, R51, R52, R53, R54, R55, R56, R57, R58, R59, R61, R62, R63, R64, R65, R66, R88, R89, R90, R91, R92, R93, R94, R95: 10K, symbol Device:R
- added R36, R37, R38, R39, R40, R41, R42, R43, R44, R45, R46, R47, R48, R60, R67, R68, R69, R70, R71, R76, R77, R82: 220, symbol Device:R
- added R72, R73, R74, R75: 680, symbol Device:R
- added R78, R79, R80, R81: 47, symbol Device:R
- added R83, R84: 75, symbol Device:R
- added R85, R86, R87: 1K, symbol Device:R
- added SW10: DSIC10LSGET, lcsc:SW-SMD_20P-L26.4-W6.2-P2.54-LS9.8, symbol LCSC:DSIC10LSGET
- added SW2, SW3, SW4, SW5, SW6, SW7, SW8, SW9: TS-1088-AR02016, lcsc:SW-SMD_L3.9-W3.0-P4.45, symbol LCSC:TS-1088-AR02016
- added U10: ~, symbol my:MC7REV2
- added U14: BME280, lcsc:LGA-8_BME280_BL, symbol LCSC:BME280
- added U15: S322527M20PF10PPM, lcsc:CRYSTAL-SMD_4P-L3.2-W2.5-BL, symbol LCSC:S322527M20PF10PPM
- added U16: TXB0108RGYR, lcsc:VQFN-20_L4.5-W3.5-P0.50-BL-EP, symbol LCSC:TXB0108RGYR
- added U17: TX5813, my:TX5813, symbol my:TX5813_1
- C11, C14, C15: value 0.1uF -> 100nF
- CN3: footprint lcsc:CONN-TH_S3B-ZR-SM4A-TF-LF-SN -> LCSC:CONN-TH_S3B-ZR-SM4A-TF-LF-SN
- R17, R18, R19, R20, R21, R22: value 33 -> 220
- R4: value 1K -> 220
- R5: value 1K -> 680
- R6: value 1K -> 10K
- U13: value 100UF -> 100uF
Connections:
- net +12V: now also J1.1 (Pin_1), J1.2 (Pin_2), J1.3 (Pin_3), J1.4 (Pin_4), J1.5 (Pin_5), J1.6 (Pin_6), LED14.2 (A)
- net +3.3V: now also Card1.4 (VDD), R6.2, SW1.2, U2.10 (CLKSEL0), U2.28 (VDDIO), U2.3 (VDD), U2.5 (PS1), U3.1 (VDDIO), U3.10 (VDD), C29.1, C30.1, C32.2, C33.2, C34.2, LED16.2 (A), LED4.1 (A), LED5.1 (A), LED6.1 (A), LED7.1 (A), LED8.1 (A), LED9.1 (A), R25.2, R26.2, R27.1, R58.2, R59.2, R61.2, R62.2, R63.2, R64.2, R65.2, R66.2, SW10.14 (B5), SW10.15 (B4), SW10.16 (B3), SW10.17 (B2), SW10.18 (B1), SW10.19, SW10.20, SW2.2, SW3.2, SW4.2, SW5.2, SW6.2, SW7.2, SW8.2, SW9.2, U14.2 (CSB), U14.6 (VDDIO), U14.8 (VDD), U16.10 (OE), U16.2 (VCCA)
- net +5V: now also CN3.1, U5.21 (AVDD), U5.24 (PVDD), U5.3 (DVDD), C36.2, C37.2, C38.2, J10.1 (Pin_1), J9.2 (Pin_2), LED15.2 (A), R85.2, R86.2, R87.2, R88.2, U10.17 (5V), U10.18 (5V), U10.19 (5V), U10.20 (5V), U10.21 (5V), U10.22 (5V), U10.23 (5V), U10.24 (SBUS3), U16.19 (VCCB), U17.10 (VCC)
- net GND: now also CN3.2, CN3.4, CN3.5, Card1.12, Card1.13, Card1.3 (Vss1), Card1.6 (Vss2), R4.2, R5.2, U2.2 (GND), U2.25 (GND), U2.26 (XOUT32/CLKSEL1), U3.3 (VSS), U3.5 (SDO), U3.6 (CSB), U3.8 (VSS), U3.9 (VSS), U5.20 (AGND), U5.4 (DGND), C28.1, C29.2, C30.2, C31.1, C32.1, C33.1, C34.1, C35.2, C36.1, C37.1, C39.2, C40.1, J10.2 (Pin_2), J5.3 (Pin_3), J6.3 (Pin_3), J7.3 (Pin_3), J8.3 (Pin_3), NT1.3, NT2.2, Q10.2 (S), Q7.2 (S), Q8.2 (S), Q9.2 (S), R24.2, R28.1, R35.1, R49.2, R50.2, R51.2, R52.2, R53.2, R54.2, R55.2, R56.2, R57.2, R72.2, R73.2, R74.2, R75.2, R76.2, R77.2, R78.2, R79.2, R80.2, R81.2, R82.2, R83.2, R89.1, R90.1, R91.1, R92.1, R93.1, R94.1, R95.1, SW10.10 (B9), SW10.8 (A8), SW10.9 (A9), U10.10 (GND), U10.11 (GND), U10.12 (GND), U10.13 (GND), U10.14 (GND), U10.15 (GND), U10.16 (SBUS2), U10.9 (GND), U14.1 (GND), U14.7 (GND), U15.2 (GND), U15.4 (GND), U16.11 (GND), U16.21 (EP), U17.11 (GND), U17.9 (GND); no longer R4.1, R5.1, R6.1, U9.10 (PGND)
- net INA_ALERT: now also R6.1, LED3.2 (A); no longer R6.2
- net INA_SCL: no longer R5.2
- net INA_SDA: no longer R4.2
- net LED1_POWER: now also J2.1 (Pin_1), R67.2
- net LED2_POWER: now also J2.2 (Pin_2), R60.2
- net LED3_POWER: now also J2.3 (Pin_3), R68.2
- net LED4_POWER: now also J2.4 (Pin_4), R69.2
- net LED5_POWER: now also J2.5 (Pin_5), R70.2
- net LED6_POWER: now also J2.6 (Pin_6), R71.2
- net PGND: now also U5.23 (PGND), U9.10 (PGND), C38.1, NT1.2, R29.1, R30.1, R31.1, R32.1, R33.1, R34.1; no longer CN1.2 (+), CN1.3, CN1.4, CN2.1, CN2.2, CN2.4 (-), CN4.1, CN4.2, CN4.4 (-), CN5.1, CN5.2, CN5.4 (-), CN6.1, CN6.2, CN6.4 (-), P1.2
- net VBAT: now also CN1.2 (+), LED11.2 (A), R23.1; no longer CN1.1 (-)
- net VBUS: now also C35.1, LED2.2 (A)
- net VMOTORS: now also LED12.2 (A)
- net VSYS: now also LED13.2 (A)
- net at Q6.4 (G), R22.1: now also R33.2
- net at Q5.4 (G), R21.1: now also R31.2
- net at U6.1: now also U6.2, U17.1 (AGND)
- net at U6.3: now also U6.4, NT2.1, U17.3 (AGND)
- net at U6.5: now also U17.2 (ANT)
- net BNO580_NRST: now reaches U2.11 (NRST)
- net BNO580_INTN: now reaches U2.14 (H_INTN)
- net at U2.15 (ENV_SCL): now also R26.1, U14.4 (SCK)
- net at U2.16 (ENV_SDA): now also R25.1, U14.3 (SDI)
- net BNO580_MOSI: now reaches U2.17 (SA0/H_MOSI)
- net BNO580_CSN: now reaches U2.18 (H_CSN)
- net BNO580_SCLK: now reaches U2.19 (H_SCL/SCK/RX)
- net BNO580_MISO: now reaches U2.20 (H_SDA/H_MISO/TX)
- net BNO580_BOOTN: now reaches U2.4 (BOOTN)
- net BNO580_BOOTN: now also R27.2
- net BNO580_WAKE: now reaches U2.6 (PS0/WAKE)
- net at U2.9 (CAP): now also C31.2
- net at Q3.4 (G), R19.1: now also R34.2
- net BMP580_SCK: now reaches U3.2 (SCK)
- net BMP580_SDI: now reaches U3.4 (SDI)
- net BMP580_INT: now reaches U3.7 (INT)
- net at Q4.4 (G), R20.1: now also R32.2
- net at Q1.4 (G), R17.1: now also R29.2
- net VIDEO: now reaches CN3.3
- net VIDEO: now also J10.3 (Pin_3), R84.1
- net SD_DAT3: now reaches Card1.1 (CD/DAT3)
- net SD_DAT3: now also R66.1
- net SD_CMD: now reaches Card1.2 (CMD)
- net SD_CMD: now also R65.1
- net SD_CLK: now reaches Card1.5 (CLK)
- net SD_CLK: now also R64.1
- net SD_DAT0: now reaches Card1.7 (DAT0)
- net SD_DAT0: now also R63.1
- net SD_DAT1: now reaches Card1.8 (DAT1)
- net SD_DAT1: now also R62.1
- net SD_DAT2: now reaches Card1.9 (DAT2)
- net SD_DAT2: now also R61.1
- net SD_CD: now reaches Card1.CD
- net SD_CD: now also R58.1
- net SD_WP: now reaches Card1.WP
- net SD_WP: now also R59.1
- net at LED1.1 (DIG1): now also Q7.3 (D)
- net at LED1.10 (G): now also R43.1
- net at LED1.11 (D2D1): now also R41.1
- net at LED1.12 (DIG2): now also Q10.3 (D)
- net at LED1.13 (F): now also R45.1
- net at LED1.14 (A): now also R42.1
- net at LED1.2 (D): now also LED1.7 (D), R39.1
- net at LED1.3 (DP): now also R40.1
- net at LED1.4 (E): now also R37.1
- net at LED1.5 (DIG3): now also Q8.3 (D)
- net at LED1.6 (C): now also R38.1
- net at LED1.8 (B): now also R44.1
- net at LED1.9 (DIG4): now also Q9.3 (D)
- net at Q2.4 (G), R18.1: now also R30.2
- net BUTTON_LEFT: now reaches SW1.1
- net BUTTON_LEFT: now also R49.1
- net MAX7456_SCLK_5V: now reaches U5.10 (SCLK)
- net MAX7456_SCLK_5V: now also U16.12 (B8)
- net MAX7456_SDOUT_5V: now reaches U5.11 (SDOUT)
- net MAX7456_SDOUT_5V: now also U16.14 (B6)
- net MAX7456_LOS_5V: now reaches U5.12 (LOS)
- net MAX7456_LOS_5V: now also R86.1, U16.17 (B3)
- net MAX7456_VSYNC_5V: now reaches U5.17 (~{VSYNC})
- net MAX7456_VSYNC_5V: now also R85.1
- net MAX7456_HSYNC_5V: now reaches U5.18 (~{HSYNC})
- net MAX7456_HSYNC_5V: now also R87.1
- net MAX7456_RESET_5V: now reaches U5.19 (~{RESET})
- net MAX7456_RESET_5V: now also R88.1, U16.18 (B2)
- net at U5.22 (VIN): now also C41.2
- net at U5.25 (SAG): now also C43.1
- net at U5.26 (VOUT): now also C42.1
- net XTAL1: now reaches U5.5 (CLKIN)
- net XTAL1: now also C40.2, U15.3
- net XTAL2: now reaches U5.6 (XFB)
- net XTAL2: now also C39.1, U15.1
- net MAX7456_CS: now reaches U5.8 (~{CS})
- net MAX7456_SDIN_5V: now reaches U5.9 (SDIN)
- net MAX7456_SDIN_5V: now also U16.13 (B7)
- net TPS_ENABLE: now reaches U7.1 (EN/UVLO)
- net TPS_ENABLE: now also R28.2
- net TPS_ADDRESS: now reaches U7.2 (MODE)
- net TPS_ADDRESS: now also R35.2
- net TPS_SCL: now reaches U7.3 (SCL)
- net TPS_SDA: now reaches U7.4 (SDA)
- new net: D4.2 (A), J6.2 (Pin_2)
- new net: C42.2, C43.2, R84.2
- new net: LED5.2 (K), R60.1
- new net: LED3.1 (K), R4.1
- new net: LED12.1 (K), R73.1
- new net: Q7.1 (G), R46.2
- new net: LED15.1 (K), R76.1
- new net: LED2.1 (K), R72.1
- new net: LED8.2 (K), R70.1
- new net: LED18.1 (K), R80.1
- new net: LED17.1 (K), R79.1
- new net: D3.2 (A), J5.2 (Pin_2)
- new net: LED6.2 (K), R68.1
- new net: LED19.1 (K), R81.1
- new net: LED16.1 (K), R77.1, R82.1
- new net: LED4.2 (K), R67.1
- new net: CN1.1 (-), CN1.3, CN1.4, NT1.1, P1.2
- new net: LED14.1 (K), R75.1
- new net: D3.1 (K), D4.1 (K), D5.1 (K), D6.1 (K), J9.1 (Pin_1)
- new net: D6.2 (A), J8.2 (Pin_2)
- new net: D5.2 (A), J7.2 (Pin_2)
- new net: Q9.1 (G), R47.2
- new net: Q10.1 (G), R48.2
- new net: LED10.1 (K), R78.1
- new net: Q8.1 (G), R36.2
- new net: LED11.1 (K), R5.1
- new net: LED13.1 (K), R74.1
- new net: LED7.2 (K), R69.1
- new net: LED9.2 (K), R71.1
- new net BUTTON_DECREASE: R52.1, SW4.1
- new net BUTTON_F1: R54.1, SW6.1
- new net BUTTON_F2: R55.1, SW7.1
- new net BUTTON_F3: R56.1, SW8.1
- new net BUTTON_F4: R57.1, SW9.1
- new net BUTTON_INCREASE: R51.1, SW3.1
- new net BUTTON_OK: R53.1, SW5.1
- new net BUTTON_RIGHT: R50.1, SW2.1
- new net DIP_1: R89.2, SW10.1 (A1)
- new net DIP_2: R90.2, SW10.2 (A2)
- new net DIP_3: R91.2, SW10.3 (A3)
- new net DIP_4: R92.2, SW10.4 (A4)
- new net DIP_5: R93.2, SW10.5 (A5)
- new net DIP_6: R94.2, SW10.6 (A6)
- new net DIP_7: R95.2, SW10.7 (A7)
- new net DISP_A: R41.2
- new net DISP_B: R44.2
- new net DISP_C: R38.2
- new net DISP_D: R39.2
- new net DISP_D2D1: R45.2
- new net DISP_DIG1: R46.1
- new net DISP_DIG2: R48.1
- new net DISP_DIG3: R36.1
- new net DISP_DIG4: R47.1
- new net DISP_DP: R40.2
- new net DISP_E: R37.2
- new net DISP_F: R42.2
- new net DISP_G: R43.2
- new net MAX7456_LOS_3.3V: U16.4 (A3)
- new net MAX7456_RESET_3.3V: U16.3 (A2)
- new net MAX7456_SCLK_3.3V: U16.9 (A8)
- new net MAX7456_SDIN_3.3V: U16.8 (A7)
- new net MAX7456_SDOUT_3.3V: U16.7 (A6)
- new net MGND: CN2.1, CN2.2, CN2.4 (-), CN4.1, CN4.2, CN4.4 (-), CN5.1, CN5.2, CN5.4 (-), CN6.1, CN6.2, CN6.4 (-), NT1.4
- new net MOTOR1_LED: LED10.2 (A)
- new net MOTOR2_LED: LED17.2 (A)
- new net MOTOR3_LED: LED18.2 (A)
- new net MOTOR4_LED: LED19.2 (A)
- new net MOTOR_PWM1: J5.1 (Pin_1)
- new net MOTOR_PWM2: J6.1 (Pin_1)
- new net MOTOR_PWM3: J7.1 (Pin_1)
- new net MOTOR_PWM4: J8.1 (Pin_1)
- new net RADIO_PWM1: U10.1 (CH1)
- new net RADIO_PWM2: U10.2 (CH2)
- new net RADIO_PWM3: U10.3 (CH3)
- new net RADIO_PWM4: U10.4 (CH4)
- new net RADIO_PWM5: U10.5 (CH5)
- new net RADIO_PWM6: U10.6 (CH6)
- new net RADIO_PWM7: U10.7 (CH7)
- new net VIDEO_OSD: C41.1, R83.1, U17.7 (VIDEO)
- new net VOLTAGE_MONITOR_ADC: C28.2, R23.2, R24.1
- new net VTX_CH1: SW10.11 (B8), U17.6 (CH1)
- new net VTX_CH2: SW10.12 (B7), U17.5 (CH2)
- new net VTX_CH3: SW10.13 (B6), U17.4 (CH3)
- no-connect marks 2 -> 23
Other:
- note added: "+12V Regulator"
- note added: "+3.3V Regulator"
- note added: "+5V Regulator"
- note added: "BMP580 Barometric"
- note added: "BNO080 IMU"
- note added: "Buttons"
- note added: "Camera Conn"
- note added: "Channel LEDs"
- note added: "Crystal"
- note added: "DIP Switches"
- note added: "Data Voltage Shifter"
- note added: "Display"
- note added: "IMPORTANT: For redundancy, as many power sources available as possible are taken and used. To monitor power usage throughout flight, the VBAT runs through the INA226 power monitor, then goes to motors WITHOUT a diode. (Otherwise diodes would have to drop ~30A worth of 0.7V) The ESC PWM 5V outputs also provide the option of latching onto the +5V line with a solder connection incase the 5V regulato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"
- note added: "LED Channels"
- note added: "Motor PWMs"
- note added: "Motor Power"
- note added: "Motor and Voltage LEDs"
- note added: "Net Tie"
- note added: "OSD Injector"
- note added: "Radio Reciever"
- note added: "SD Card"
- note added: "USB C"
- note added: "VIDEO Circuitry"
- note added: "VTX and SMA Conn"
- note added: "Voltage/Current Monitor"
- moved on the sheet: CN1, CN2, CN4, CN5, CN6, Card1, LED1, U1, U11, U12, U2, U3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

Commit message: Update
Parts:
- removed C42, C43: C_Polarized, symbol Device:C_Polarized
- removed CN3: Camera Conn, LCSC:CONN-TH_S3B-ZR-SM4A-TF-LF-SN, symbol LCSC:S3B-ZR-SM4A-TF(LF)(SN)
- removed Card1: SD-006M, LCSC:SD-SMD_SD-006M, symbol LCSC:SD-006M
- removed J1, J2, J3, J4: Conn_01x06_Pin, symbol Connector:Conn_01x06_Pin
- removed LED10, LED17, LED18, LED19: KT-0603B, lcsc:LED0603-RD, symbol LCSC:Bluelight0603
- removed LED8, LED9: KT-0603W, lcsc:LED0603-R-RD_WHITE, symbol LCSC:0603Whitelight_C2290
- removed NT1: NetTie_4, symbol Device:NetTie_4
- removed P1: WJ127-5.0-2P, LCSC:CONN-TH_2P-P5.00_CPC3703CTR, symbol LCSC:WJ127-5.0-2P
- removed Q4, Q6: CSD16340Q3, LCSC:VSON-CLIP-8_L3.3-W3.3-P0.65-BL, symbol LCSC:CSD16340Q3
- removed R57, R59, R89, R90, R91, R92, R93, R94, R95: 10K, symbol Device:R
- removed R70, R71: 220, symbol Device:R
- removed R79, R80, R81: 47, symbol Device:R
- removed SW10: DSIC10LSGET, lcsc:SW-SMD_20P-L26.4-W6.2-P2.54-LS9.8, symbol LCSC:DSIC10LSGET
- added BUZ1: CPT-9019S-SMT-TR, LCSC:BUZ-SMD_L9.0-W9.0-P8.00-LS9.3, symbol LCSC:CPT-9019S-SMT-TR
- added C42, C66, C74: RVT1C220M0405_C3356_22uF, LCSC:CAP-SMD_BD4.0-L4.3-W4.3-FD-LS5.3, symbol LCSC:RVT1C220M0405_C3356
- added C43, C56, C68, C77: 10uF, Capacitor_SMD:C_0402_1005Metric, symbol Device:C
- added C44, C45, C46, C47, C48, C49, C50, C51, C63, C64, C67, C78: 100nF, Capacitor_SMD:C_0402_1005Metric, symbol Device:C
- added C52, C53, C54, C55, C65: 1uF, Capacitor_SMD:C_0402_1005Metric, symbol Device:C
- added C57, C58: 2.2uF, Capacitor_SMD:C_0402_1005Metric, symbol Device:C
- added C59, C62: 6.8pF, Capacitor_SMD:C_0402_1005Metric, symbol Device:C
- added C60, C61: 20pF, Capacitor_SMD:C_0402_1005Metric, symbol Device:C
- added C69, C75, C76: 0.1uF, Capacitor_SMD:C_0402_1005Metric, symbol Device:C
- added C70: 15nF, Capacitor_SMD:C_0402_1005Metric, symbol Device:C
- added C71: 3.3nF, Capacitor_SMD:C_0402_1005Metric, symbol Device:C
- added C72: 10nF, Capacitor_SMD:C_0402_1005Metric, symbol Device:C
- added C73: 150pF, Capacitor_SMD:C_0402_1005Metric, symbol Device:C
- added Card2: TF-01A, LCSC:TF-SMD_TF-01A, symbol LCSC:TF-01A
- added J1: Conn_02x07_Odd_Even, Connector_PinHeader_2.54mm:PinHeader_2x07_P2.54mm_Vertical, symbol Connector_Generic:Conn_02x07_Odd_Even
- added J12: Conn_02x02_Top_Bottom, Connector_PinHeader_2.54mm:PinHeader_2x02_P2.54mm_Vertical, symbol Connector_Generic:Conn_02x02_Top_Bottom
- added J13, J18: Conn_01x14_Pin, Connector_PinHeader_2.54mm:PinHeader_1x14_P2.54mm_Vertical, symbol Connector:Conn_01x14_Pin
- added J14, J19: Conn_01x06_Pin, Connector_PinHeader_2.54mm:PinHeader_1x06_P2.54mm_Vertical, symbol Connector:Conn_01x06_Pin
- added J15, J20: Conn_01x14_Socket, Connector_PinSocket_2.54mm:PinSocket_1x14_P2.54mm_Vertical, symbol Connector:Conn_01x14_Socket
- added J16, J17: Conn_01x06_Socket, Connector_PinSocket_2.54mm:PinSocket_1x06_P2.54mm_Vertical, symbol Connector:Conn_01x06_Socket
- added J2: Conn_01x02_Pin, Connector_PinHeader_1.00mm:PinHeader_1x02_P1.00mm_Vertical, symbol Connector:Conn_01x02_Pin
- added J21: Conn_02x04_Odd_Even, Connector_PinHeader_2.54mm:PinHeader_2x04_P2.54mm_Vertical, symbol Connector_Generic:Conn_02x04_Odd_Even
- added L2: FCM1608KF-601T03, LCSC:L0603, symbol LCSC:FCM1608KF-601T03
- added LED8: KT-0603R, LCSC:LED0603-RD, symbol LCSC:KT-0603R
- added LED9: KT-0603YG, LCSC:LED0603-RD, symbol LCSC:XL-0603QYGC
- added NT1, NT10, NT11, NT12, NT13, NT14, NT15, NT16, NT7, NT8, NT9: NetTie_2, NetTie:NetTie-2_THT_Pad0.3mm, symbol Device:NetTie_2
- added NT17: NetTie_2, NetTie:NetTie-2_THT_Pad1.0mm, symbol Device:NetTie_2
- added R100, R103, R104, R99: 4.7K, Resistor_SMD:R_0402_1005Metric, symbol Device:R
- added R101: 10K, Resistor_SMD:R_0603_1608Metric, symbol Device:R
- added R102, R96, R97, R98: 10K, Resistor_SMD:R_0402_1005Metric, symbol Device:R
- added SW10, SW14: DSIC03LSGET, LCSC:SW-SMD_DSIC03LSGET, symbol LCSC:DSIC03LSGET
- added SW11, SW12: TS-1088-AR02016, LCSC:SW-SMD_L3.9-W3.0-P4.45, symbol LCSC:TS-1088-AR02016
- added SW13: MK-11C04-G013, LCSC:SW-SMD_MK-11C04-G013, symbol LCSC:MK-11C04-G013
- added U18: 100uF, LCSC:CAP-SMD_BD6.3-L6.6-W6.6-LS7.2-FD-1, symbol LCSC:RVT1E101M0607100UF25V
- added U19: TPS259850RQPR, LCSC:QFN-26_L5.0-W4.5_TPS259850RQPR, symbol LCSC:TPS259850RQPR
- added U20: LD1117D33TR, LCSC:SO-8_L4.9-W3.9-P1.27-LS6.0-BL, symbol LCSC:LD1117D33TR
- added X1: X322525MOB4SI, LCSC:CRYSTAL-SMD_4P-L3.2-W2.5-BL, symbol LCSC:X322525MOB4SI
- added X2: Q13FC1350000400, LCSC:FC-135R_L3.2-W1.5, symbol LCSC:Q13FC1350000400
- C10, C11, C14, C15, C16, C17, C18, C19, C20, C21, C22, C23, C24, C26, C27, C29, C30, C31, C32, C33, C34, C35, C36, C37, C38, C39, C40, C41: footprint (none) -> Capacitor_SMD:C_0402_1005Metric
- C12, C13: footprint (none) -> Capacitor_SMD:C_0603_1608Metric
- C25: footprint lcsc:CAP-SMD_BD6.3-L6.6-W6.6-LS7.2-FD -> LCSC:CAP-SMD_BD6.3-L6.6-W6.6-LS7.2-FD
- C28: footprint Capacitor_SMD:C_0603_1608Metric -> Capacitor_SMD:C_0402_1005Metric
- J10, J5, J6, J7, J8: footprint (none) -> Connector_PinHeader_2.54mm:PinHeader_1x03_P2.54mm_Vertical
- J9: footprint (none) -> Connector_PinHeader_1.00mm:PinHeader_1x02_P1.00mm_Vertical
- LED11, LED12, LED13, LED14, LED15, LED16, LED2, LED3: footprint lcsc:LED0603-RD -> LCSC:LED0603-RD
- LED4, LED5, LED6, LED7: footprint lcsc:LED0603-R-RD_WHITE -> LCSC:LED0603-R-RD_WHITE
- NT2: footprint (none) -> NetTie:NetTie-2_THT_Pad1.0mm
- Q10, Q7, Q8, Q9: footprint lcsc:SOT-23_L2.9-W1.3-P1.90-LS2.4-BR -> LCSC:SOT-23_L2.9-W1.3-P1.90-LS2.4-BR
- R1, R10, R11, R12, R13, R14, R16, R17, R18, R19, R2, R21, R25, R26, R27, R28, R29, R30, R31, R34, R35, R36, R37, R38, R39, R4, R40, R41, R42, R43, R44, R45, R46, R47, R48, R49, R5, R58, R6, R60, R61, R62, R63, R64, R65, R66, R67, R68, R69, R7, R72, R73, R74, R75, R76, R77, R8, R82, R85, R86, R87, R88, R9: footprint (none) -> Resistor_SMD:R_0402_1005Metric
- R15: footprint lcsc:R2512 -> LCSC:R2512
- R20, R22: value 220 -> 10K; footprint (none) -> Resistor_SMD:R_0402_1005Metric
- R23, R24: footprint Resistor_SMD:R_0603_1608Metric -> Resistor_SMD:R_0402_1005Metric
- R32, R54: value 10K -> 1K; footprint (none) -> Resistor_SMD:R_0402_1005Metric
- R33: value 10K -> 68K; footprint (none) -> Resistor_SMD:R_0402_1005Metric
- R50: value 10K -> 160; footprint (none) -> Resistor_SMD:R_0402_1005Metric
- R51: value 10K -> 1.1K; footprint (none) -> Resistor_SMD:R_0402_1005Metric
- R52: value 10K -> 48K; footprint (none) -> Resistor_SMD:R_0402_1005Metric
- R53: value 10K -> 1.5K; footprint (none) -> Resistor_SMD:R_0402_1005Metric
- R55: value 10K -> 2.2K; footprint (none) -> Resistor_SMD:R_0402_1005Metric
- R56: value 10K -> 50K; footprint (none) -> Resistor_SMD:R_0402_1005Metric
- R78: value 47 -> 100; footprint (none) -> Resistor_SMD:R_0402_1005Metric
- R83, R84: footprint (none) -> Resistor_SMD:R_0603_1608Metric
- SW1, SW2, SW3, SW4, SW5, SW6, SW7, SW8, SW9: footprint lcsc:SW-SMD_L3.9-W3.0-P4.45 -> LCSC:SW-SMD_L3.9-W3.0-P4.45
- U10: footprint (none) -> my:MC7RE
- U13: footprint lcsc:CAP-SMD_BD6.3-L6.6-W6.6-LS7.2-FD-1 -> LCSC:CAP-SMD_BD6.3-L6.6-W6.6-LS7.2-FD-1
- U14: footprint lcsc:LGA-8_BME280_BL -> LCSC:LGA-8_BME280_BL
- U15: footprint lcsc:CRYSTAL-SMD_4P-L3.2-W2.5-BL -> LCSC:CRYSTAL-SMD_4P-L3.2-W2.5-BL
- U16: footprint lcsc:VQFN-20_L4.5-W3.5-P0.50-BL-EP -> LCSC:VQFN-20_L4.5-W3.5-P0.50-BL-EP
- U4: footprint lcsc:IND-SMD_L5.5-W5.3 -> LCSC:IND-SMD_L5.5-W5.3
- U6: footprint lcsc:SMA-TH_SMA-KWE_C7498154 -> LCSC:SMA-TH_SMA-KWE_C7498154
- U7: footprint lcsc:VQFN-21_L5.0-W3.0-P0.50-TL -> LCSC:VQFN-21_L5.0-W3.0-P0.50-TL
- U8: footprint lcsc:IND-SMD_L7.5-W7.2-1 -> LCSC:IND-SMD_L7.5-W7.2-1
- USB1: footprint lcsc:USB-C-SMD_TYPE-C16PIN_C668624 -> LCSC:USB-C-SMD_TYPE-C16PIN_C668624
Connections:
- net BMP580_SCK is gone; now on net MAIN_SCK_T: U3.2 (SCK)
- net BMP580_SDI is gone; now on net MAIN_SDA_T: U3.4 (SDI)
- net LED5_PWM is gone; now on net GND_B: R20.2
- net LED6_PWM is gone; now on net GND: R22.2
- net MAX7456_CS is gone; now on net MAX7456_CS_5V: U5.8 (~{CS})
- net TPS_SCL is gone; now on net MAIN_SCK_B: U7.3 (SCL)
- net TPS_SDA is gone; now on net MAIN_SDA_B: U7.4 (SDA)
- net +12V: now also J1.2 (Pin_2), J1.4 (Pin_4), J13.10 (Pin_10); no longer C26.1, R11.2, R15.2, U7.13 (ISN)
- net +3.3V: now also R9.2, U1.100 (VDD), U1.11 (VDD), U1.20 (VREF+), U1.27 (VDD), U1.50 (VDD), U1.6 (VBAT), U1.75 (VDD), C42.1, C43.1, C45.1, C46.1, C47.1, C48.1, C49.1, C50.1, C51.1, C52.1, C53.1, C54.1, C55.1, C56.1, C64.1, C65.1, C67.1, C68.1, Card2.4 (VDD), J1.10 (Pin_10), J1.12 (Pin_12), J13.12 (Pin_12), J14.1 (Pin_1), L2.2, R100.1, R102.1, R103.2, R104.2, R96.1, R97.1, R98.1, R99.1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; no longer C1.2, LED4.1 (A), LED5.1 (A), LED6.1 (A), LED7.1 (A), R9.1, U11.6 (VS+), U16.10 (OE), U16.2 (VCCA), U2.10 (CLKSEL0)
- net +5V: now also J1.6 (Pin_6), J1.8 (Pin_8), J13.11 (Pin_11), J2.2 (Pin_2); no longer C36.2, C37.2, C38.2, C6.2, C7.2, C8.2, C9.2, J10.1 (Pin_1), R8.2, R85.2, R86.2, R87.2, R88.2, U16.19 (VCCB), U17.10 (VCC), U5.21 (AVDD), U5.24 (PVDD), U5.3 (DVDD), U9.5 (FB), U9.7 (VOUT)
- net BMP580_INT: now also U1.96 (PB9), R102.2
- net BNO580_BOOTN: now also U1.34 (PB0)
- net BNO580_CSN: now also U1.77 (PA15)
- net BNO580_INTN: now also U1.33 (PC5), R98.2
- net BNO580_MISO: now also U1.30 (PA6)
- net BNO580_MOSI: now also U1.31 (PA7)
- net BNO580_NRST: now also U1.32 (PC4), R97.2
- net BNO580_SCLK: now also U1.29 (PA5)
- net BNO580_WAKE: now also U1.35 (PB1), R96.2
- net BUTTON_DECREASE: now also U1.39 (PE9); no longer R52.1
- net BUTTON_F1: now also U1.41 (PE11); no longer R54.1
- net BUTTON_F2: now also U1.42 (PE12); no longer R55.1
- net BUTTON_F3: now also U1.43 (PE13); no longer R56.1
- net BUTTON_F4: now also U1.51 (PB12)
- net BUTTON_INCREASE: now also U1.38 (PE8); no longer R51.1
- net BUTTON_LEFT: now also U1.36 (PB2); no longer R49.1
- net BUTTON_OK: now also U1.40 (PE10); no longer R53.1
- net BUTTON_RIGHT: now also U1.37 (PE7); no longer R50.1
- net DIP_1: now also U1.52 (PB13), SW10.6 (B1)
- net DIP_2: now also U1.54 (PB15), SW10.5 (B2)
- net DIP_3: now also U1.55 (PD8), SW10.4 (B3)
- net DISP_A: now also U1.87 (PD6)
- net DISP_B: now also U1.86 (PD5)
- net DISP_C: now also U1.85 (PD4)
- net DISP_D: now also U1.84 (PD3)
- net DISP_D2D1: now also U1.58 (PD11)
- net DISP_DIG1: now also U1.91 (PB5)
- net DISP_DIG2: now also U1.90 (PB4)
- net DISP_DIG3: now also U1.89 (PB3)
- net DISP_DIG4: now also U1.88 (PD7)
- net DISP_DP: now also U1.67 (PA8)
- net DISP_E: now also U1.72 (PA13)
- net DISP_F: now also U1.69 (PA10)
- net DISP_G: now also U1.68 (PA9)
- net GND: now also C12.1, C13.1, U1.10 (VSS), U1.19 (VSSA), U1.26 (VSS), U1.49 (VSS), U1.74 (VSS), U1.99 (VSS), BUZ1.2 (-), C42.2, C43.2, C45.2, C46.2, C47.2, C48.2, C49.2, C50.2, C51.2, C52.2, C53.2, C54.2, C55.2, C56.2, C57.1, C58.1, C59.2, C60.2, C61.1, C62.2, C63.2, C64.2, C65.2, C67.2, C68.2, C77.2, C78.2, Card2.10 (GND), Card2.11 (GND), Card2.12 (GND), Card2.13 (GND)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; no longer C1.1, C17.1, C18.1, C2.2, C23.1, C24.1, C28.1, C3.1, C36.1, C37.1, C39.2, C4.1, C40.1, C5.1, C6.1, C7.1, C8.1, C9.1, J10.2 (Pin_2), NT2.2, R13.1, R14.2, R16.1, R24.2, R28.1, R35.1, R49.2, R50.2, R51.2, R52.2, R53.2, R54.2, R55.2, R56.2, R78.2, R83.2, U11.1 (A1), U11.2 (A0), U11.7 (GND), U15.2 (GND)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
- net LED1_POWER: now also J21.8 (Pin_8)
- net LED2_POWER: now also J21.6 (Pin_6)
- net LED3_POWER: now also J21.4 (Pin_4)
- net LED4_POWER: now also J21.2 (Pin_2)
- net MOTOR_PWM1: now also U1.22 (PA0)
- net MOTOR_PWM2: now also U1.23 (PA1)
- net MOTOR_PWM3: now also U1.24 (PA2)
- net MOTOR_PWM4: now also U1.25 (PA3)
- net RADIO_PWM1: now also U1.64 (PC7)
- net RADIO_PWM2: now also U1.63 (PC6)
- net RADIO_PWM3: now also U1.62 (PD15)
- net RADIO_PWM4: now also U1.61 (PD14)
- net RADIO_PWM5: now also U1.60 (PD13)
- net RADIO_PWM6: now also U1.59 (PD12)
- net SD_CD: now also U1.82 (PD1), Card2.9 (CD)
- net SD_CLK: now also U1.80 (PC12), Card2.5 (CLK(SCLK))
- net SD_CMD: now also U1.83 (PD2), Card2.3 (CMD(DI))
- net SD_DAT0: now also U1.65 (PC8), Card2.7 (DAT0(D0))
- net SD_DAT1: now also U1.66 (PC9), Card2.8 (DAT1(RSV))
- net SD_DAT2: now also U1.78 (PC10), Card2.1 (DAT2(RSV))
- net SD_DAT3: now also U1.79 (PC11), Card2.2 (CDDAT3(CS))
- net USB_DN: now also U1.70 (PA11)
- net USB_DP: now also U1.71 (PA12)
- net VBAT: now also J13.8 (Pin_8); no longer CN1.2 (+), R23.1, R3.2, U11.10 (VIN+), U11.8 (VBUS)
- net VBUS: now also C77.1
- net VMOTORS: now also J13.9 (Pin_9); no longer CN2.3 (+), CN4.3 (+), CN5.3 (+), CN6.3 (+), D2.2 (A), R3.1, U11.9 (VIN-)
- net VSYS: now also C78.1, J1.1 (Pin_1), J1.3 (Pin_3), J1.5 (Pin_5), J1.7 (Pin_7), J13.13 (Pin_13), J18.10 (Pin_10), J18.11 (Pin_11), J18.12 (Pin_12), J18.13 (Pin_13), J18.14 (Pin_14), J18.7 (Pin_7), J18.8 (Pin_8), J18.9 (Pin_9); no longer C16.2, C27.2, C3.2, C4.2, C5.2, D2.1 (K), R7.1, U13.2, U7.7 (VIN), U9.12 (VIN)
- net VTX_CH1: now also SW14.4 (B3)
- net VTX_CH2: now also SW14.5 (B2)
- net VTX_CH3: now also SW14.6 (B1)
- net at U5.25 (SAG): now also C66.1
- net at R84.2: now also C66.2, U18.1
- net at C31.2, U2.9 (CAP): now also U2.10 (CLKSEL0)
- net at R33.2: now also CN1.2 (+), R32.2, R55.1, C75.2, LED8.2 (A), U19.23 (VIN), U19.24 (VIN), U19.25 (VIN), U19.26 (VIN), U20.4 (VIN); no longer R22.1
- net +5V_B: now reaches C17.2, U7.18 (VCC)
- net +5V_B: now also C6.2, C7.2, C8.2, C9.2, R8.2, R85.2, R86.2, R87.2, R88.2, U16.19 (VCCB), U9.5 (FB), U9.7 (VOUT), J15.11 (Pin_11), SW13.1
- net at U5.26 (VOUT): now also U18.2
- net at U17.1 (AGND), U6.1, U6.2: now also NT2.1, U17.3 (AGND), U6.3, U6.4, NT17.1
- net MGND_B: now reaches CN1.1 (-), CN1.3, CN1.4
- net MGND_B: now also C1.1, C28.1, CN2.2, CN2.3 (+), CN2.4 (-), CN4.2, CN4.3 (+), CN4.4 (-), CN5.2, CN5.3 (+), CN5.4 (-), CN6.2, CN6.3 (+), CN6.4 (-), R24.2, R49.1, R50.1, R51.2, R52.2, U11.1 (A1), U11.2 (A0), U11.7 (GND), C69.1, C70.2, C71.2, C72.1, C73.1, C74.2, C75.1, C76.2, LED9.1 (K), NT1.2, NT10.2, NT11.2, NT12.2, NT13.2, NT14.2, NT15.2, NT16.2, NT7.2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
- net at D5.1 (K), D6.1 (K), J9.1 (Pin_1): no longer D3.1 (K), D4.1 (K)
- net MAX7456_CS_5V: now reaches U16.15 (B5)
- net MAX7456_CS_3.3V_B: now reaches U16.6 (A5)
- net MAX7456_CS_3.3V_B: now also J20.4 (Pin_4)
- net BUZZER: now reaches R78.1
- net BUZZER: now also U1.53 (PB14)
- net at R20.1: now also U7.21 (EXTVCC); no longer R32.2
- net MAX7456_SCLK_3.3V_T: now reaches U1.1 (PE2)
- net MAX7456_SCLK_3.3V_T: now also J18.1 (Pin_1)
- net HSE_IN: now reaches U1.12 (PH0)
- net HSE_IN: now also C61.2, X1.1 (OSC1)
- net HSE_OUT: now reaches U1.13 (PH1)
- net HSE_OUT: now also C60.1, X1.3 (OSC2)
- net RESET: now reaches U1.14 (NRST)
- net RESET: now also C63.1, SW11.2
- net LED1_PWM_T: now reaches U1.15 (PC0)
- net LED1_PWM_T: now also J13.1 (Pin_1)
- net LED2_PWM_T: now reaches U1.16 (PC1)
- net LED2_PWM_T: now also J13.2 (Pin_2)
- net LED3_PWM_T: now reaches U1.17 (PC2)
- net LED3_PWM_T: now also J13.3 (Pin_3)
- net LED4_PWM_T: now reaches U1.18 (PC3)
- net LED4_PWM_T: now also J13.4 (Pin_4)
- net MAX7456_LOS_3.3V_T: now reaches U1.2 (PE3)
- net MAX7456_LOS_3.3V_T: now also J18.5 (Pin_5)
- net at U1.21 (VDDA): now also L2.1
- net VOLTAGE_ADC_T: now reaches U1.28 (PA4)
- net VOLTAGE_ADC_T: now also J14.5 (Pin_5)
- net MAX7456_CS_3.3V_T: now reaches U1.3 (PE4)
- net MAX7456_CS_3.3V_T: now also J18.4 (Pin_4)
- net MAX7456_SDOUT_3.3V_T: now reaches U1.4 (PE5)
- net MAX7456_SDOUT_3.3V_T: now also J18.3 (Pin_3)
- net EXTRA_I2C_EN: now reaches U1.44 (PE14)
- net EXTRA_I2C_EN: now also J12.4 (Pin_4)
- net EXTRA_I2C_INT: now reaches U1.45 (PE15)
- net EXTRA_I2C_INT: now also J12.3 (Pin_3)
- net EXTRA_I2C_SCL: now reaches U1.46 (PB10)
- net EXTRA_I2C_SCL: now also J12.1 (Pin_1), R103.1
- net EXTRA_I2C_SDA: now reaches U1.47 (PB11)
- net EXTRA_I2C_SDA: now also J12.2 (Pin_2), R104.1
- net at U1.48 (VCAP_1): now also C57.2
- net MAX7456_SDIN_3.3V_T: now reaches U1.5 (PE6)
- net MAX7456_SDIN_3.3V_T: now also J18.2 (Pin_2)
- net at U1.73 (VCAP_2): now also C58.2
- net LSE_IN: now reaches U1.8 (PC14)
- net LSE_IN: now also C59.1, X2.1
- net LSE_OUT: now reaches U1.9 (PC15)
- net LSE_OUT: now also C62.1, X2.2
- net MAIN_SCK_T: now reaches U1.92 (PB6)
- net MAIN_SCK_T: now also J13.6 (Pin_6), J14.2 (Pin_2), R99.2
- net MAIN_SDA_T: now reaches U1.93 (PB7)
- net MAIN_SDA_T: now also J13.7 (Pin_7), J14.3 (Pin_3), R100.2
- net BOOT: now reaches U1.94 (BOOT0)
- net BOOT: now also R22.1, SW12.2
- net INA_ALERT_T: now reaches U1.95 (PB8)
- net INA_ALERT_T: now also LED3.2 (A), R6.1, J14.4 (Pin_4)
- net TPS_ENABLE_T: now reaches U1.97 (PE0)
- net TPS_ENABLE_T: now also J13.5 (Pin_5)
- net MAX7456_RESET_3.3V_T: now reaches U1.98 (PE1)
- net MAX7456_RESET_3.3V_T: now also J18.6 (Pin_6)
- net GND_B: now reaches U5.29 (EP)
- net GND_B: now also C16.1, C17.1, C18.1, C19.1, C2.2, C20.1, C21.1, C22.1, C23.1, C24.1, C25.1, C27.1, C3.1, C36.1, C37.1, C38.1, C39.2, C4.1, C40.1, C5.1, C6.1, C7.1, C8.1, C9.1, J10.2 (Pin_2), NT2.2, Q1.1 (S), Q1.2 (S), Q1.3 (S), Q2.1 (S), Q2.2 (S), Q2.3 (S), Q3.1 (S), Q3.2 (S), Q3.3 (S), Q5.1 (S), Q5.2 (S), Q5.3 (S), R13.1, R14.2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
- removed net INA_ALERT: LED3.2 (A), R6.1, U11.3 (Alert)
- net INA_SCL renamed MAIN_SCK_B
- net MAIN_SCK_B: now also J15.6 (Pin_6), J16.2 (Pin_2)
- net INA_SDA renamed MAIN_SDA_B
- net MAIN_SDA_B: now also J15.7 (Pin_7), J16.3 (Pin_3)
- net LED1_PWM renamed LED1_PWM_B
- net LED1_PWM_B: now also J15.1 (Pin_1)
- net LED2_PWM renamed LED2_PWM_B
- net LED2_PWM_B: now also J15.2 (Pin_2)
- net LED3_PWM renamed LED3_PWM_B
- net LED3_PWM_B: now also J15.3 (Pin_3)
- net LED4_PWM renamed LED4_PWM_B
- net LED4_PWM_B: now also J15.4 (Pin_4)
- net MAX7456_LOS_3.3V renamed MAX7456_LOS_3.3V_B
- net MAX7456_LOS_3.3V_B: now also J20.5 (Pin_5)
- net MAX7456_RESET_3.3V renamed MAX7456_RESET_3.3V_B
- net MAX7456_RESET_3.3V_B: now also J20.6 (Pin_6)
- net MAX7456_SCLK_3.3V renamed MAX7456_SCLK_3.3V_B
- net MAX7456_SCLK_3.3V_B: now also J20.1 (Pin_1)
- net MAX7456_SDIN_3.3V renamed MAX7456_SDIN_3.3V_B
- net MAX7456_SDIN_3.3V_B: now also J20.2 (Pin_2)
- net MAX7456_SDOUT_3.3V renamed MAX7456_SDOUT_3.3V_B
- net MAX7456_SDOUT_3.3V_B: now also J20.3 (Pin_3)
- removed net MGND: CN2.1, CN2.2, CN2.4 (-), CN4.1, CN4.2, CN4.4 (-), CN5.1, CN5.2, CN5.4 (-), CN6.1, CN6.2, CN6.4 (-)
- removed net PGND: C16.1, C19.1, C20.1, C21.1, C22.1, C25.1, C27.1, C38.1, Q1.1 (S), Q1.2 (S), Q1.3 (S), Q2.1 (S), Q2.2 (S), Q2.3 (S), Q3.1 (S), Q3.2 (S), Q3.3 (S), Q5.1 (S), Q5.2 (S), Q5.3 (S), R29.1, R30.1, R31.1, R32.1, R33.1, R34.1, U13.1, U5.23 (PGND), U7.9 (PGND), U9.10 (PGND)
- net RADIO_PWM7: no longer names the net of U10.7 (CH7)
- net TPS_ADDRESS: no longer names the net of R35.2, U7.2 (MODE)
- net TPS_ADDRESS: now also C44.1
- net TPS_ENABLE renamed TPS_ENABLE_B
- net TPS_ENABLE_B: now also J15.5 (Pin_5)
- net VIDEO renamed VIDEO_IN
- net VIDEO_IN: now also C41.1, R83.1; no longer R84.1
- removed net VIDEO_OSD: C41.1, R83.1, U17.7 (VIDEO)
- net VOLTAGE_MONITOR_ADC renamed VOLTAGE_ADC_B
- net VOLTAGE_ADC_B: now also J16.5 (Pin_5)
- new net: C69.2, R32.1, U19.22 (VDD)
- new net: C73.2, R52.1, U19.9 (IREF)
- new net: C72.2, R51.1, U19.7 (IMON)
- new net: R10.1, R9.1, U12.4 (FB)
- new net: C76.1, R56.1, U20.2 (VOUT), U20.3 (VOUT), U20.6 (VOUT), U20.7 (VOUT)
- new net: D3.1 (K), D4.1 (K), J2.1 (Pin_1)
- new net: BUZ1.1 (+), R78.2
- new net: R33.1, R49.2, U19.18 (EN/UVLO)
- new net: R54.2, R55.2, U19.19 (PG)
- new net: R56.2, U19.21 (SWEN)
- new net: LED8.1 (K), R53.1
- new net: R50.2, U19.8 (ILIM)
- new net: C70.1, U19.6 (ITIMER)
- new net: R53.2, U19.20 (~{FLT})
- new net: C71.1, U19.4 (DVDT)
- new net: LED9.2 (A), R54.1
- new net +12V_B: C26.1, J15.10 (Pin_10), J21.1 (Pin_1), J21.3 (Pin_3), J21.5 (Pin_5), J21.7 (Pin_7), R11.2, R15.2, U7.13 (ISN)
- new net +3.3V_B: C1.2, J15.12 (Pin_12), J16.1 (Pin_1), LED4.1 (A), LED5.1 (A), LED6.1 (A), LED7.1 (A), R101.2, R28.1, U11.6 (VS+), U16.10 (OE), U16.2 (VCCA)
- new net INA_ALERT_B: J16.4 (Pin_4), R101.1, U11.3 (Alert)
- new net VBAT_B: C74.1, J15.8 (Pin_8), R23.1, R3.2, U11.10 (VIN+), U11.8 (VBUS), U19.10 (VOUT), U19.11 (VOUT), U19.12 (VOUT), U19.13 (VOUT)
- new net VIDEO_OUT: R84.1, U17.7 (VIDEO)
- new net VMOTORS_B: CN2.1, CN4.1, CN5.1, CN6.1, D2.2 (A), J15.9 (Pin_9), R3.1, U11.9 (VIN-)
- new net VSYS_B: C16.2, C27.2, C3.2, C4.2, C5.2, D2.1 (K), J15.13 (Pin_13), J20.10 (Pin_10), J20.11 (Pin_11), J20.12 (Pin_12), J20.13 (Pin_13), J20.14 (Pin_14), J20.7 (Pin_7), J20.8 (Pin_8), J20.9 (Pin_9), R7.1, U13.2, U7.7 (VIN), U9.12 (VIN)
- new net VTX_SUPPLY: C36.2, C37.2, C38.2, J10.1 (Pin_1), SW13.C, U17.10 (VCC), U5.21 (AVDD), U5.24 (PVDD), U5.3 (DVDD)
- no-connect marks 23 -> 44
Other:
- note added: "Buzzer"
- note added: "Extra I2C"
- note added: "Extra V Rails"
- note added: "POWER"
- note added: "STM32F7"
- note added: "Voltage LEDs"
- note removed: "Camera Conn"
- note removed: "Channel LEDs"
- note removed: "Motor and Voltage LEDs"
- note removed: "Net Tie"
- moved on the sheet: J5, J6, J7, J8, J9, LED1, U1, U10, U11, U12, U2, U3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
