File: PCB/Controller/Controller.kicad_sch (KiCad schematic)
At the start: 274 parts, among them CN1 XT60PW_M, CN2 XT60PW_F, CN4 XT60PW_F, CN5 XT60PW_F, CN6 XT60PW_F, J1 Conn_02x07_Odd_Even, J10 Conn_01x03_Pin, J12 Conn_02x02_Top_Bottom, J13 Conn_01x14_Pin, J14 Conn_01x06_Pin, J15 Conn_01x14_Socket, J16 Conn_01x06_Socket, J17 Conn_01x06_Socket, J18 Conn_01x14_Pin, J19 Conn_01x06_Pin, J2 Conn_01x02_Pin, J20 Conn_01x14_Socket, J21 Conn_02x04_Odd_Even, J5 Conn_01x03_Pin, J6 Conn_01x03_Pin, J7 Conn_01x03_Pin, J8 Conn_01x03_Pin, J9 Conn_01x02_Pin, Q1 CSD16340Q3, Q10 LBSS138LT1G, Q2 CSD16340Q3, Q3 CSD16340Q3, Q5 CSD16340Q3, Q7 LBSS138LT1G, Q8 LBSS138LT1G, Q9 LBSS138LT1G, SW1 TS-1088-AR02016, SW10 DSIC03LSGET, SW11 TS-1088-AR02016, SW12 TS-1088-AR02016, SW13 MK-11C04-G013, SW14 DSIC03LSGET, SW2 TS-1088-AR02016, SW3 TS-1088-AR02016, SW4 TS-1088-AR02016, SW5 TS-1088-AR02016, SW6 TS-1088-AR02016, SW7 TS-1088-AR02016, SW8 TS-1088-AR02016, SW9 TS-1088-AR02016, U1 STM32F765VGTx, U11 INA226AQDGSRQ1, U12 LMR51430, U13 100uF, U14 BME280, U15 S322527M20PF10PPM, U16 TXB0108RGYR, U17 TX5813, U18 100uF, U19 TPS259850RQPR, U2 BNO080, U20 LD1117D33TR, U3 BMP580, U4 XAL5050-562MEC, U5 MAX7456EUI, U6 SMA_Conn, U7 TPS55289RYQR, U8 XAL7070-472MEC, U9 TPS630701RNMT, X1 X322525MOB4SI, X2 Q13FC1350000400

Commit message: Update
Parts:
- added B1: CR2032-BS-6-1, lcsc:BAT-TH_CR2032-BS-6-1, symbol LCSC:CR2032-BS-6-1
- added B2: CR2032-BS-5-1, lcsc:BAT-TH_CR2032-BS-5-1, symbol LCSC:CR2032-BS-5-1
- added BT1: BH-18650-B1BA002, lcsc:BATTERY-SMD_18650-1S-L77.1-W20.7-1, symbol LCSC:BH-18650-B1BA002
- added C100: 33uF, Capacitor_SMD:C_0603_1608Metric, symbol Device:C
- added C101, C103, C85, C87, C92, C94, C97: 10uF, Capacitor_SMD:C_0603_1608Metric, symbol Device:C
- added C102, C98: 22uF, Capacitor_SMD:C_0603_1608Metric, symbol Device:C
- added C104, C105, C110, C111, C113, C115, C117, C119, C79, C80: 0.1uF, Capacitor_SMD:C_0402_1005Metric, symbol Device:C
- added C106, C95: 20pF, Capacitor_SMD:C_0402_1005Metric, symbol Device:C
- added C107: 220nF, Capacitor_SMD:C_0603_1608Metric, symbol Device:C
- added C108, C109, C112, C114, C116, C118, C120, C81, C82: 10uF, Capacitor_SMD:C_0402_1005Metric, symbol Device:C
- added C83, C84: 10uF, Capacitor_SMD:C_0805_2012Metric, symbol Device:C
- added C86: 100nF, Capacitor_SMD:C_0402_1005Metric, symbol Device:C
- added C88, C89, C90: 22uF, Capacitor_SMD:C_0805_2012Metric, symbol Device:C
- added C91, C93: 100nF, Capacitor_SMD:C_0603_1608Metric, symbol Device:C
- added C96: 1uF, Capacitor_SMD:C_0402_1005Metric, symbol Device:C
- added C99: 4.7uF, Capacitor_SMD:C_0603_1608Metric, symbol Device:C
- added CM1: RX5808, lcsc:COMM-SMD_12P_RX5808, symbol LCSC:RX5808
- added D10: Diode, Diode_SMD:D_SMB, symbol Device:D
- added J11: Conn_01x10_Pin, Connector_PinHeader_2.54mm:PinHeader_1x10_P2.54mm_Vertical, symbol Connector:Conn_01x10_Pin
- added J3: Conn_01x40_Socket, Connector_FFC-FPC:Hirose_FH12-40S-0.5SH_1x40-1MP_P0.50mm_Horizontal, symbol Connector:Conn_01x40_Socket
- added J4: Conn_01x06_Pin, Connector_PinHeader_2.54mm:PinHeader_1x06_P2.54mm_Vertical, symbol Connector:Conn_01x06_Pin
- added L3: XFL4020-152MEC, LCSC:IND-SMD_L4.0-W4.0-A, symbol LCSC:XFL4020-152MEC
- added L4: 22uH, LCSC:IND-SMD_L5.8-W5.8, symbol Device:L_Ferrite
- added LED10, LED17, LED18, LED19, LED20, LED21, LED22: KT-0603YG, LCSC:LED0603-RD, symbol LCSC:XL-0603QYGC
- added LED23: KT-0603YR, LCSC:LED0603-RD, symbol LCSC:XL-0603QYGC
- added R105: 396K, Resistor_SMD:R_0402_1005Metric, symbol Device:R
- added R106, R70, R81, R89, R91, R92, R95: 10K, Resistor_SMD:R_0402_1005Metric, symbol Device:R
- added R107, R109, R110, R80: 4.7K, Resistor_SMD:R_0402_1005Metric, symbol Device:R
- added R108: 2.2K, Resistor_SMD:R_0402_1005Metric, symbol Device:R
- added R111, R112, R113: 1.5K, Resistor_SMD:R_0402_1005Metric, symbol Device:R
- added R114: 3.3K, Resistor_SMD:R_0402_1005Metric, symbol Device:R
- added R115: 1.5k, Resistor_SMD:R_0402_1005Metric, symbol Device:R
- added R116, R90: 220, Resistor_SMD:R_0402_1005Metric, symbol Device:R
- added R57, R59: 5.1K, Resistor_SMD:R_0402_1005Metric, symbol Device:R
- added R71: 100K, Resistor_SMD:R_0402_1005Metric, symbol Device:R
- added R79: 80, Resistor_SMD:R_0402_1005Metric, symbol Device:R
- added R93: 1.8K, Resistor_SMD:R_0402_1005Metric, symbol Device:R
- added R94: 1K, Resistor_SMD:R_0402_1005Metric, symbol Device:R
- added RV1: 10K, Potentiometer_SMD:Potentiometer_Bourns_3314J_Vertical, symbol Device:R_Potentiometer
- added SW15: DSIC03LSGET, LCSC:SW-SMD_DSIC03LSGET, symbol LCSC:DSIC03LSGET
- added SW16, SW17: SW_Push, Button_Switch_SMD:SW_Push_1P1T-SH_NO_CK_KMR2xxG, symbol Switch:SW_Push
- added SW18: K3-1204D-L, lcsc:SW-TH_K3-1204D-L, symbol LCSC:K3-1204D-L
- added U22: ~, Package_DFN_QFN:QFN-48-1EP_7x7mm_P0.5mm_EP5.6x5.6mm_ThermalVias, symbol my:TW8819
- added U23: ESP32-S3-MINI-1U, RF_Module:ESP32-S2-MINI-1U, symbol RF_Module:ESP32-S3-MINI-1U
- added U24: TPS630701RNMT, LCSC:VQFN-15_L3.0-W2.5-P0.50-BL, symbol LCSC:TPS630701RNMT
- added U25: BQ21088YBGR, lcsc:DSBGA-8_L1.5-W1.0-R2-C4-P0.40-BL, symbol LCSC:BQ21088YBGR
- added U26: L80RE-M37, lcsc:GPSM-SMD_12P-L16.0-W16.0-P2.54-BL, symbol LCSC:L80RE-M37
- added U27: LD1117S33TR_SOT223, Package_TO_SOT_SMD:SOT-223-3_TabPin2, symbol Regulator_Linear:LD1117S33TR_SOT223
- added U28: CAT4104, LCSC:SOIC-8_L4.9-W3.9-P1.27-LS6.0-BL, symbol My_Library:CAT4104
- added U29: MT3608, Package_TO_SOT_SMD:SOT-23-6, symbol Regulator_Switching:MT3608
- added U30: SMA_Conn, LCSC:SMA-TH_SMA-KWE_C7498154, symbol LCSC:SMA-KWE_C7498154
- added U31: LD1117S18TR_SOT223, Package_TO_SOT_SMD:SOT-223-3_TabPin2, symbol Regulator_Linear:LD1117S18TR_SOT223
- added USB2: TYPE-C 16P(073), LCSC:USB-C-SMD_TYPE-C16PIN_C668624, symbol LCSC:TYPE-C16P(073)
- added X3: X322527MSB4SI, lcsc:CRYSTAL-SMD_4P-L3.2-W2.5-BL-1, symbol LCSC:X322527MSB4SI
- U12: value LMR51430 -> LMR51430XF
Connections:
- net +3.3V: now also C120.2, C80.2, U26.10 (RESET), U26.4 (VCC)
- net DIP_3: now also U1.57 (PD10); no longer U1.55 (PD8)
- net GND: now also B1.2, C120.1, C79.1, C80.1, C96.1, SW16.2, SW17.2, U26.12 (GND), U26.3 (GND)
- net GPS_TX: now reaches U1.56 (PD9)
- net GPS_TX: now also U26.2 (TXD1)
- net EXTRA_I2C_INT: no longer names the net of J12.3 (Pin_3)
- net EXTRA_I2C_INT: no longer U1.45 (PE15)
- new net: LED17.1 (K), R112.1
- new net: LED19.1 (K), R114.1
- new net: R93.1, RV1.3
- new net: LED23.1 (K), R90.1
- new net: CM1.9 (RSSI), R108.1
- new net: D10.2 (A), L4.2, U29.1 (SW)
- new net: C100.1, SW18.1, U25.B2 (SYS)
- new net: LED21.1 (K), R116.1
- new net: CM1.2 (ANT), U30.5
- new net: CM1.4 (CH1), SW15.6 (B1)
- new net: CM1.5 (CH2), SW15.5 (B2)
- new net: CM1.6 (CH3), SW15.4 (B3)
- new net: R105.2, R95.1, U29.3 (FB)
- new net: R57.1, USB2.A5 (CC1)
- new net: LED10.1 (K), R111.1
- new net: C86.1, U24.3 (VAUX)
- new net: B1.1, C79.2, U26.5 (V_BCKP)
- new net: L3.1, U24.11 (L1)
- new net: L3.2, U24.9 (L2)
- new net: LED18.1 (K), R113.1
- new net: J11.1 (Pin_1), U23.28 (IO33)
- new net: J11.2 (Pin_2), U23.29 (IO34)
- new net: J11.3 (Pin_3), U23.31 (IO35)
- new net: J11.4 (Pin_4), U23.32 (IO36)
- new net: J11.5 (Pin_5), U23.33 (IO37)
- new net: J11.6 (Pin_6), U23.34 (IO38)
- new net: J11.7 (Pin_7), U23.35 (IO39)
- new net: J11.8 (Pin_8), U23.36 (IO40)
- new net: J11.9 (Pin_9), U23.37 (IO41)
- new net: J11.10 (Pin_10), U23.38 (IO42)
- new net: R70.2, U24.1 (PS/S), U24.14 (EN)
- new net: R71.1, U24.2 (PG)
- new net: R106.1, U25.D1 (TS/MR)
- new net: R79.2, U22.10 (XTI)
- new net: C107.2, U22.2 (DIAG0/YIN0+/YIN1)
- new net: LED20.1 (K), R115.1
- new net: R93.2, U28.8 (RSET)
- new net: R59.1, USB2.B5 (CC2)
- new net: R94.1, U28.6 (EN/PWM)
- new net +1.8V_R: C108.1, C111.1, C112.2, C113.2, C116.2, C117.2, C94.2, LED22.2 (A), U22.1 (AVDAD), U22.22 (VDD18), U22.42 (VDD18), U22.47 (AVDPLL), U31.2 (VO)
- new net +24V_R: C98.2, D10.1 (K), J3.2 (Pin_2), J4.1 (Pin_1), LED19.2 (A), R105.1
- new net +3.3V_R: C102.1, C103.1, C104.1, C105.1, C109.2, C110.2, C114.1, C115.1, C92.2, J3.4 (Pin_4), J4.3 (Pin_3), LED21.2 (A), R109.1, R110.1, R80.1, R81.2, R89.1, U22.18 (VDD33), U22.37 (VDD33), U23.3 (3V3), U27.2 (VO)
- new net +5V_R: C118.1, C119.1, C87.2, C88.2, C89.2, C90.2, C91.2, CM1.8 (+5V), J4.2 (Pin_2), LED20.2 (A), R71.2, R94.2, U24.5 (FB), U24.7 (VOUT), U27.3 (VI), U28.7 (VIN)
- new net B0: J3.21 (Pin_21), U22.17 (PWM1/TRSPB/FPB0)
- new net B1: J3.22 (Pin_22), U22.19 (PWM2/CSPR/FPB1)
- new net B2: J3.23 (Pin_23), U22.40 (FPB2)
- new net B3: J3.24 (Pin_24), U22.41 (FPB3)
- new net B4: J3.25 (Pin_25), U22.43 (FPB4)
- new net B5: J3.26 (Pin_26), U22.44 (FPB5)
- new net B6: J3.27 (Pin_27), U22.45 (FPB6)
- new net B7: J3.28 (Pin_28), U22.46 (FPB7)
- new net BOOT0_R: R89.2, SW17.1, U23.4 (IO0)
- new net BQ_INT: U23.27 (IO47), U25.A1 (~{INT})
- new net DE: J3.34 (Pin_34), U22.16 (TROE/sDE/FPDE)
- new net DISP: J3.31 (Pin_31), R80.2, U23.16 (IO12)
- new net DIVIDER_R: R91.2, R92.1, U23.21 (IO17)
- new net EN_R: C96.2, R81.1, SW16.1, U23.45 (EN)
- new net G0: J3.13 (Pin_13), U22.20 (GPIO1/TCLP/FPG0)
- new net G1: J3.14 (Pin_14), U22.21 (GPIO2/TRUD/FPG1)
- new net G2: J3.15 (Pin_15), U22.32 (FPG2/sD1)
- new net G3: J3.16 (Pin_16), U22.33 (FPG3/sD0)
- new net G4: J3.17 (Pin_17), U22.34 (FPG4)
- new net G5: J3.18 (Pin_18), U22.35 (FPG5)
- new net G6: J3.19 (Pin_19), U22.38 (FPG6)
- new net G7: J3.20 (Pin_20), U22.39 (FPG7)
- new net GND_R: BT1.1, C100.2, C101.2, C102.2, C103.2, C104.2, C105.2, C106.2, C108.2, C109.1, C110.1, C111.2, C112.1, C113.1, C114.2, C115.2, C116.1, C117.1, C118.2, C119.2, C81.2, C82.2, C83.1, C84.1, C85.1, C86.2, C87.1, C88.1, C89.1, C90.1, C91.1, C92.1, C93.1, C94.1, C95.1, C97.1, C98.1, C99.2, CM1.1 (GND), CM1.12 (GND), CM1.3 (GND), CM1.7 (GND), J3.29 (Pin_29), J3.3 (Pin_3), J3.36 (Pin_36), J4.6 (Pin_6), LED22.1 (K), R106.2, R107.2, R111.2, R112.2, R113.2, R114.2, R115.2, R116.2, R57.2, R59.2, R90.2, R91.1, R95.2, RV1.2, SW15.1 (A1), SW15.2 (A2), SW15.3 (A3), U22.25 (VSS), U22.3 (DIAG1/YIN0-/YIN1), U22.36 (VSS), U22.4 (DIAG2/YIN2+/YIN2), U22.48 (AVSPLL), U22.5 (DIAG3/YIN2-/YIN3), U22.6 (AVSAD), U23.1 (GND), U23.2 (GND), U23.42 (GND), U23.43 (GND), U23.46 (GND), U23.47 (GND), U23.48 (GND), U23.49 (GND), U23.50 (GND), U23.51 (GND), U23.52 (GND), U23.53 (GND), U23.54 (GND), U23.55 (GND), U23.56 (GND), U23.57 (GND), U23.58 (GND), U23.59 (GND), U23.60 (GND), U23.61 (GND), U23.62 (GND), U23.63 (GND), U23.64 (GND), U23.65 (GND), U24.10 (PGND), U24.15 (VSEL), U24.4 (GND), U24.6 (FB2), U25.D2 (GND), U27.1 (GND), U28.5 (GND), U29.2 (GND), U30.1, U30.2, U30.3, U30.4, U31.1 (GND), USB2.1 (SHELL), USB2.2 (SHELL), USB2.3 (SHELL), USB2.4 (SHELL), USB2.A1B12 (GND), USB2.B1A12 (GND), X3.2 (GND), X3.4 (GND)
- new net GPIO_LED: LED23.2 (A), U23.25 (IO21)
- new net GPS_JAM_T: U1.45 (PE15)
- new net GPS_RX: U1.55 (PD8), U26.1 (RXD1)
- new net HSE_IN_R: C106.1, R79.1, X3.3 (OSC2)
- new net HSE_OUT_R: C95.2, U22.11 (XTO), X3.1 (OSC1)
- new net HSYNC: J3.32 (Pin_32), U22.15 (TCSPL/sHS/FPHS)
- new net PCLK: J3.30 (Pin_30), U22.13 (TCCLK/sCLK/FPCLK)
- new net R0: J3.5 (Pin_5), U22.23 (GPIO3/TRCLK/FPR0)
- new net R1: J3.6 (Pin_6), U22.24 (GPIO4/TCLRL/FPR1)
- new net R2: J3.7 (Pin_7), U22.26 (FPR2/sD7)
- new net R3: J3.8 (Pin_8), U22.27 (FPR3/sD6)
- new net R4: J3.9 (Pin_9), U22.28 (FPR4/sD5)
- new net R5: J3.10 (Pin_10), U22.29 (FPR5/sD4)
- new net R6: J3.11 (Pin_11), U22.30 (FPR6/sD3)
- new net R7: J3.12 (Pin_12), U22.31 (FPR7/sD2)
- new net RESET_TW8819: U22.7 (RSTB), U23.26 (IO26)
- new net RSSI: R107.1, R108.2, U23.30 (IO48)
- new net SCL_R: J4.5 (Pin_5), R109.2, U22.9 (SCL), U23.9 (IO5), U25.B1 (SCL)
- new net SDA_R: J4.4 (Pin_4), R110.2, U22.8 (SDA), U23.8 (IO4), U25.C1 (SDA)
- new net USB_DN_R: U23.23 (USB_D-), USB2.A7 (DN1), USB2.B7 (DN2)
- new net USB_DP_R: U23.24 (USB_D+), USB2.A6 (DP1), USB2.B6 (DP2)
- new net VBAT_R: BT1.2, C101.1, LED17.2 (A), R92.2, U25.C2 (BAT)
- new net VBUS_R: C81.1, C82.1, C99.1, LED10.2 (A), U25.A2 (IN), USB2.A4B9 (VBUS), USB2.B4A9 (VBUS)
- new net VIDEO_R: C107.1, CM1.11 (VIDEO)
- new net VLED-: J3.1 (Pin_1), U28.1 (LED1)
- new net VSYNC: J3.33 (Pin_33), U22.14 (TRSPT/sVS/FPVS)
- new net VSYS_R: C83.2, C84.2, C85.2, C93.2, C97.2, L4.1, LED18.2 (A), R70.1, SW18.2, U24.12 (VIN), U29.4 (EN), U29.5 (IN), U31.3 (VI)
- new net XL: J3.39 (Pin_39), U23.19 (IO15)
- new net XR: J3.37 (Pin_37), U23.17 (IO13)
- new net YD: J3.38 (Pin_38), U23.18 (IO14)
- new net YU: J3.40 (Pin_40), U23.20 (IO16)
- no-connect marks 44 -> 72
Other:
- note added: "3.3V/1.8V regulators"
- note added: "Backlight Circuitry"
- note added: "Battery Holder"
- note added: "Boot Pushbuttons"
- note added: "Decoupling"
- note added: "GPS"
- note added: "LED Current Sink Driver"
- note added: "RX5808 Circuitry"
- note added: "Reciever PCB For TFT Display"
- note added: "Status LEDs"
- note added: "TFT Display"
- note added: "TFT Display Conn"
- note added: "TW8819 Circuitry"
- note added: "Troubleshoot Header"
- note added: "USB C and Bat Charger"
- note added: "Voltage Booster for Backlight"
- moved on the sheet: BUZ1, C66, CN1, CN2, CN4, CN5, CN6, Card2, J1, J12, J2, J5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

Commit message: Update
Parts:
- removed B1: CR2032-BS-6-1, lcsc:BAT-TH_CR2032-BS-6-1, symbol LCSC:CR2032-BS-6-1
- removed B2: CR2032-BS-5-1, lcsc:BAT-TH_CR2032-BS-5-1, symbol LCSC:CR2032-BS-5-1
- removed BT1: BH-18650-B1BA002, lcsc:BATTERY-SMD_18650-1S-L77.1-W20.7-1, symbol LCSC:BH-18650-B1BA002
- removed C100: 33uF, Capacitor_SMD:C_0603_1608Metric, symbol Device:C
- removed C101, C103, C85, C87, C92, C94, C97: 10uF, Capacitor_SMD:C_0603_1608Metric, symbol Device:C
- removed C102, C98: 22uF, Capacitor_SMD:C_0603_1608Metric, symbol Device:C
- removed C104, C105, C110, C111, C113, C115, C117, C119, C79, C80: 0.1uF, Capacitor_SMD:C_0402_1005Metric, symbol Device:C
- removed C106, C95: 20pF, Capacitor_SMD:C_0402_1005Metric, symbol Device:C
- removed C107: 220nF, Capacitor_SMD:C_0603_1608Metric, symbol Device:C
- removed C108, C109, C112, C114, C116, C118, C120, C81, C82: 10uF, Capacitor_SMD:C_0402_1005Metric, symbol Device:C
- removed C83, C84: 10uF, Capacitor_SMD:C_0805_2012Metric, symbol Device:C
- removed C86: 100nF, Capacitor_SMD:C_0402_1005Metric, symbol Device:C
- removed C88, C89, C90: 22uF, Capacitor_SMD:C_0805_2012Metric, symbol Device:C
- removed C91, C93: 100nF, Capacitor_SMD:C_0603_1608Metric, symbol Device:C
- removed C96: 1uF, Capacitor_SMD:C_0402_1005Metric, symbol Device:C
- removed C99: 4.7uF, Capacitor_SMD:C_0603_1608Metric, symbol Device:C
- removed CM1: RX5808, lcsc:COMM-SMD_12P_RX5808, symbol LCSC:RX5808
- removed D10: Diode, Diode_SMD:D_SMB, symbol Device:D
- removed J11: Conn_01x10_Pin, Connector_PinHeader_2.54mm:PinHeader_1x10_P2.54mm_Vertical, symbol Connector:Conn_01x10_Pin
- removed J3: Conn_01x40_Socket, Connector_FFC-FPC:Hirose_FH12-40S-0.5SH_1x40-1MP_P0.50mm_Horizontal, symbol Connector:Conn_01x40_Socket
- removed J4: Conn_01x06_Pin, Connector_PinHeader_2.54mm:PinHeader_1x06_P2.54mm_Vertical, symbol Connector:Conn_01x06_Pin
- removed L3: XFL4020-152MEC, LCSC:IND-SMD_L4.0-W4.0-A, symbol LCSC:XFL4020-152MEC
- removed L4: 22uH, LCSC:IND-SMD_L5.8-W5.8, symbol Device:L_Ferrite
- removed LED10, LED17, LED18, LED19, LED20, LED21, LED22: KT-0603YG, LCSC:LED0603-RD, symbol LCSC:XL-0603QYGC
- removed LED23: KT-0603YR, LCSC:LED0603-RD, symbol LCSC:XL-0603QYGC
- removed NT17, NT2: NetTie_2, NetTie:NetTie-2_THT_Pad1.0mm, symbol Device:NetTie_2
- removed R105: 396K, Resistor_SMD:R_0402_1005Metric, symbol Device:R
- removed R106, R70, R81, R89, R91, R92, R95: 10K, Resistor_SMD:R_0402_1005Metric, symbol Device:R
- removed R107, R109, R110, R80: 4.7K, Resistor_SMD:R_0402_1005Metric, symbol Device:R
- removed R108: 2.2K, Resistor_SMD:R_0402_1005Metric, symbol Device:R
- removed R111, R112, R113: 1.5K, Resistor_SMD:R_0402_1005Metric, symbol Device:R
- removed R114: 3.3K, Resistor_SMD:R_0402_1005Metric, symbol Device:R
- removed R115: 1.5k, Resistor_SMD:R_0402_1005Metric, symbol Device:R
- removed R116, R90: 220, Resistor_SMD:R_0402_1005Metric, symbol Device:R
- removed R57, R59: 5.1K, Resistor_SMD:R_0402_1005Metric, symbol Device:R
- removed R71: 100K, Resistor_SMD:R_0402_1005Metric, symbol Device:R
- removed R79: 80, Resistor_SMD:R_0402_1005Metric, symbol Device:R
- removed R93: 1.8K, Resistor_SMD:R_0402_1005Metric, symbol Device:R
- removed R94: 1K, Resistor_SMD:R_0402_1005Metric, symbol Device:R
- removed RV1: 10K, Potentiometer_SMD:Potentiometer_Bourns_3314J_Vertical, symbol Device:R_Potentiometer
- removed SW15: DSIC03LSGET, LCSC:SW-SMD_DSIC03LSGET, symbol LCSC:DSIC03LSGET
- removed SW16, SW17: SW_Push, Button_Switch_SMD:SW_Push_1P1T-SH_NO_CK_KMR2xxG, symbol Switch:SW_Push
- removed SW18: K3-1204D-L, lcsc:SW-TH_K3-1204D-L, symbol LCSC:K3-1204D-L
- removed U22: ~, Package_DFN_QFN:QFN-48-1EP_7x7mm_P0.5mm_EP5.6x5.6mm_ThermalVias, symbol my:TW8819
- removed U23: ESP32-S3-MINI-1U, RF_Module:ESP32-S2-MINI-1U, symbol RF_Module:ESP32-S3-MINI-1U
- removed U24: TPS630701RNMT, LCSC:VQFN-15_L3.0-W2.5-P0.50-BL, symbol LCSC:TPS630701RNMT
- removed U25: BQ21088YBGR, lcsc:DSBGA-8_L1.5-W1.0-R2-C4-P0.40-BL, symbol LCSC:BQ21088YBGR
- removed U26: L80RE-M37, lcsc:GPSM-SMD_12P-L16.0-W16.0-P2.54-BL, symbol LCSC:L80RE-M37
- removed U27: LD1117S33TR_SOT223, Package_TO_SOT_SMD:SOT-223-3_TabPin2, symbol Regulator_Linear:LD1117S33TR_SOT223
- removed U28: CAT4104, LCSC:SOIC-8_L4.9-W3.9-P1.27-LS6.0-BL, symbol My_Library:CAT4104
- removed U29: MT3608, Package_TO_SOT_SMD:SOT-23-6, symbol Regulator_Switching:MT3608
- removed U30: SMA_Conn, LCSC:SMA-TH_SMA-KWE_C7498154, symbol LCSC:SMA-KWE_C7498154
- removed U31: LD1117S18TR_SOT223, Package_TO_SOT_SMD:SOT-223-3_TabPin2, symbol Regulator_Linear:LD1117S18TR_SOT223
- removed USB2: TYPE-C 16P(073), LCSC:USB-C-SMD_TYPE-C16PIN_C668624, symbol LCSC:TYPE-C16P(073)
- removed X3: X322527MSB4SI, lcsc:CRYSTAL-SMD_4P-L3.2-W2.5-BL-1, symbol LCSC:X322527MSB4SI
Connections:
- net GND_B: now also U17.1 (AGND), U17.3 (AGND), U6.1, U6.2, U6.3, U6.4
- no-connect marks 72 -> 43
Other:
- note removed: "3.3V/1.8V regulators"
- note removed: "Backlight Circuitry"
- note removed: "Battery Holder"
- note removed: "Boot Pushbuttons"
- note removed: "Decoupling"
- note removed: "GPS"
- note removed: "LED Current Sink Driver"
- note removed: "RX5808 Circuitry"
- note removed: "Reciever PCB For TFT Display"
- note removed: "Status LEDs"
- note removed: "TFT Display"
- note removed: "TFT Display Conn"
- note removed: "TW8819 Circuitry"
- note removed: "Troubleshoot Header"
- note removed: "USB C and Bat Charger"
- note removed: "Voltage Booster for Backlight"
- moved on the sheet: Card2, USB1

Commit message: Update
Connections:
- net +5V_B: no longer C17.2, U7.18 (VCC)
- new net: C17.2, U7.18 (VCC)
Changed lines of the file:
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@@
 	)
 	(junction
+		(at 173.99 381)
+		(diameter 0)
+		(color 0 0 0 0)
+	)
+	(junction
 		(at 228.6 369.57)
 		(diameter 0)
@@
 	)
 	(junction
-		(at 153.67 115.57)
-		(diameter 0)
-		(color 0 0 0 0)
-	)
-	(junction
 		(at 237.49 173.99)
 		(diameter 0)
@@
 	(wire
 		(pts
+			(xy 173.99 381) (xy 190.5 381)
+		)
+		(stroke
+			(width 0)
+			(type default)
+		)
+	)
+	(wire
+		(pts
 			(xy 314.96 190.5) (xy 314.96 191.77)
 		)
@@
 	(wire
 		(pts
-			(xy 176.53 391.16) (xy 179.07 391.16)
-		)
-		(stroke
-			(width 0)
-			(type default)
-		)
-	)
-	(wire
-		(pts
 			(xy 119.38 314.96) (xy 128.27 314.96)
 		)
@@
 	(wire
 		(pts
-			(xy 217.17 287.02) (xy 219.71 287.02)
+			(xy 173.99 381) (xy 173.99 386.08)
 		)
 		(stroke
@@
 	(wire
 		(pts
-			(xy 370.84 378.46) (xy 369.57 378.46)
+			(xy 217.17 287.02) (xy 219.71 287.02)
 		)
 		(stroke
@@
 	(wire
 		(pts
-			(xy 200.66 250.19) (xy 200.66 271.78)
+			(xy 370.84 378.46) (xy 369.57 378.46)
 		)
 		(stroke
@@
 	(wire
 		(pts
-			(xy 434.34 185.42) (xy 452.12 185.42)
+			(xy 200.66 250.19) (xy 200.66 271.78)
 		)
 		(stroke
@@
 	(wire
 		(pts
-			(xy 466.09 81.28) (xy 461.01 81.28)
+			(xy 434.34 185.42) (xy 452.12 185.42)
 		)
 		(stroke
@@
 	(wire
 		(pts
-			(xy 449.58 259.08) (xy 452.12 259.08)
+			(xy 466.09 81.28) (xy 461.01 81.28)
 		)
 		(stroke
@@
 	(wire
 		(pts
-			(xy 200.66 271.78) (xy 205.74 271.78)
+			(xy 449.58 259.08) (xy 452.12 259.08)
 		)
 		(stroke
@@
 	(wire
 		(pts
-			(xy 176.53 381) (xy 176.53 391.16)
+			(xy 200.66 271.78) (xy 205.74 271.78)
 		)
 		(stroke
@@
 	(wire
 		(pts
-			(xy 153.67 114.3) (xy 153.67 115.57)
-		)
-		(stroke
-			(width 0)
-			(type default)
-		)
-	)
-	(wire
-		(pts
 			(xy 72.39 387.35) (xy 71.12 387.35)
 		)
@@
 	(wire
 		(pts
-			(xy 173.99 370.84) (xy 173.99 386.08)
+			(xy 173.99 370.84) (xy 173.99 381)
 		)
 		(stroke
@@
 	(wire
 		(pts
-			(xy 190.5 381) (xy 176.53 381)
-		)
-		(stroke
-			(width 0)
-			(type default)
-		)
-	)
-	(wire
-		(pts
 			(xy 55.88 302.26) (xy 54.61 302.26)
 		)
@@
 	)
 	(symbol
-		(lib_id "power:GND")
-		(at 179.07 391.16 90)
-		(unit 1)
-		(exclude_from_sim no)
-		(in_bom yes)
-		(on_board yes)
-		(dnp no)
-		(property "Reference" "#PWR0112"
-			(at 185.42 391.16 0)
-			(effects
-				(font
-					(size 1.27 1.27)
-				)
-				(hide yes)
-			)
-		)
-		(property "Value" "GND_B"
-			(at 182.118 391.16 90)
-			(effects
-				(font
-					(size 1.27 1.27)
-				)
-				(justify right)
-			)
-		)
-		(property "Footprint" ""
-			(at 179.07 391.16 0)
-			(effects
-				(font
-					(size 1.27 1.27)
-				)
-				(hide yes)
-			)
-		)
-		(property "Datasheet" ""
-			(at 179.07 391.16 0)
-			(effects
-				(font
-					(size 1.27 1.27)
-				)
-				(hide yes)
-			)
-		)
-		(property "Description" "Power symbol creates a global label with name \"GND\" , ground"
-			(at 179.07 391.16 0)
-			(effects
-				(font
-					(size 1.27 1.27)
-				)
-				(hide yes)
-			)
-		)
-		(pin "1"
-		)
-		(instances
-			(project "Controller"
-				(path "/10bda189-e6b8-4829-954f-e6c14f11b79d"
-					(reference "#PWR0112")
-					(unit 1)
-				)
-			)
-		)
-	)
-	(symbol
 		(lib_id "power:VBUS")
 		(at 191.77 314.96 90)
@@
 					(unit 1)
 				)
-			)
-		)
-	)
-	(symbol
-		(lib_id "power:VBUS")
-		(at 153.67 114.3 0)
-		(unit 1)
-		(exclude_from_sim no)
-		(in_bom yes)
-		(on_board yes)
-		(dnp no)
-		(property "Reference" "#PWR0219"
-			(at 153.67 118.11 0)
-			(effects
-				(font
-					(size 1.27 1.27)
-				)
-				(hide yes)
-			)
-		)
-		(property "Value" "+5V_B"
-			(at 150.368 109.982 0)
-			(effects
-				(font
-					(size 1.27 1.27)
-				)
-				(justify left)
-			)
-		)
-		(property "Footprint" ""
-			(at 153.67 114.3 0)
-			(effects
-				(font
-					(size 1.27 1.27)
-				)
-				(hide yes)
-			)
-		)
-		(property "Datasheet" ""
-			(at 153.67 114.3 0)
-			(effects
-				(font
-					(size 1.27 1.27)
-				)
-				(hide yes)
-			)
-		)
-		(property "Description" "Power symbol creates a global label with name \"VBUS\""
-			(at 153.67 114.3 0)
-			(effects
-				(font
-					(size 1.27 1.27)
-				)
-				(hide yes)
-			)
-		)
-		(pin "1"
-		)
-		(instances
-			(project "Controller"
-				(path "/10bda189-e6b8-4829-954f-e6c14f11b79d"
-					(reference "#PWR0219")
-					(unit 1)
-				)

Commit message: Update
Connections:
- net at L1.1: now also U9.9 (L2); no longer U9.11 (L1)
- net at L1.2: now also U9.11 (L1); no longer U9.9 (L2)
Changed lines of the file:
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@@
 		(lib_id "LCSC:XFL4020-152MEC")
 		(at 184.15 383.54 0)
+		(mirror y)
 		(unit 1)
 		(exclude_from_sim no)
@@
 		)
 		(property "Value" "XFL4020-152MEC"
-			(at 187.198 385.826 0)
+			(at 181.102 385.826 0)
 			(effects
 				(font

Commit message: Update
Parts:
- removed C26: 100nF, Capacitor_SMD:C_0402_1005Metric, symbol Device:C
- removed C66: RVT1C220M0405_C3356_22uF, LCSC:CAP-SMD_BD4.0-L4.3-W4.3-FD-LS5.3, symbol LCSC:RVT1C220M0405_C3356
- removed R15: MS122WF100MT4E, LCSC:R2512, symbol LCSC:MS122WF100MT4E
- removed U18: 100uF, LCSC:CAP-SMD_BD6.3-L6.6-W6.6-LS7.2-FD-1, symbol LCSC:RVT1E101M0607100UF25V
- added C66: 100uF, Capacitor_SMD:C_1210_3225Metric, symbol Device:C
- added C79: 22uF, Capacitor_SMD:C_1206_3216Metric, symbol Device:C
- added FPC2: FPC-05F-6PH20, lcsc:FPC-SMD_6P-P0.50_XUNPU_FPC-05F-6PH20, symbol LCSC:FPC-05F-6PH20
- added R15: 24K, Resistor_SMD:R_0402_1005Metric, symbol Device:R
- R52: value 48K -> 24K
Connections:
- net +12V_B: now also C19.2, C20.2, C21.2, C22.2, C25.2, U7.11 (VOUT), U7.12 (ISP)
- net +3.3V: now also FPC2.1, FPC2.2
- net GND: now also FPC2.3, FPC2.4, FPC2.7, FPC2.8
- net GPS_RX: now also FPC2.5
- net GPS_TX: now also FPC2.6
- net at C73.2, U19.9 (IREF): now also R15.1; no longer R52.1
- net at U5.25 (SAG): now also C79.2
- net at R84.2: now also C66.1, C79.1
- net at U5.26 (VOUT): now also C66.2
- net GPS_JAM_T: no longer names the net of U1.45 (PE15)
- new net: R15.2, R52.1
Other:
- note added: "UART FPC Port"
